File: weisse_cpu.kicad_pcb (KiCad board)
At the start: 2 copper layers, 310 x 260 mm, 30 parts

Commit message: hhhhhh
Parts:
- EINGAENGE1, LEISTUNGSNETZ1: footprint Connector_PinHeader_2.00mm:PinHeader_1x08_P2.00mm_Vertical -> Connector_PinHeader_2.54mm:PinHeader_1x08_P2.54mm_Vertical
- LAMPENSPALTEN1: footprint Connector_PinHeader_2.00mm:PinHeader_1x16_P2.00mm_Vertical -> Connector_PinHeader_2.54mm:PinHeader_1x16_P2.54mm_Vertical
- R40: footprint Resistor_THT:R_Axial_DIN0617_L17.0mm_D6.0mm_P30.48mm_Horizontal -> Resistor_THT:R_Axial_Power_L20.0mm_W6.4mm_P30.48mm
- SERVICEANZEIGE+TASTATUR1: footprint Connector_PinHeader_2.00mm:PinHeader_1x20_P2.00mm_Vertical -> Connector_PinHeader_2.54mm:PinHeader_1x20_P2.54mm_Vertical
- SIGNALNETZ1: footprint Connector_PinHeader_2.00mm:PinHeader_1x06_P2.00mm_Vertical -> Connector_PinHeader_2.54mm:PinHeader_1x06_P2.54mm_Vertical
- moved ICK11 33.7 mm to (414.3, 174.0)
- moved ICG10-1 9.11 mm to (391.3, 206.0)
- moved RM81 3.12 mm to (412.4, 206.0)
- moved ICC6 1.12 mm to (307.1, 286.0)
- moved ICD6 1.00 mm to (302.0, 265.5)
- moved ICE6 1.00 mm to (302.0, 245.0)
Routing:
- net Net-(LAMPENSPALTEN1-Pin_7): track 2.00 -> 0.00 mm
- net Net-(LAMPENSPALTEN1-Pin_5): track 2.00 -> 0.00 mm
- net Net-(LAMPENSPALTEN1-Pin_3): track 2.00 -> 0.00 mm
- net Net-(LAMPENSPALTEN1-Pin_15): track 2.00 -> 0.00 mm
- net Net-(LAMPENSPALTEN1-Pin_13): track 2.00 -> 0.00 mm
- net Net-(LAMPENSPALTEN1-Pin_11): track 2.00 -> 0.00 mm
- net Net-(LAMPENSPALTEN1-Pin_10): track 2.00 -> 0.00 mm
- net Net-(LAMPENSPALTEN1-Pin_1): track 2.00 -> 0.00 mm
Other:
- outline, holes or cut-outs redrawn

Commit message: headers
Parts:
- moved SERVICEANZEIGE+TASTATUR1 7.54 mm to (442.0, 170.5)
- moved ICH4-1 2.54 mm to (244.3, 187.0)
- moved ICK11 1.30 mm to (414.3, 175.3)
- moved RM81 0.62 mm to (411.8, 206.0)
- moved ICC6 0.50 mm to (306.6, 286.0)
- moved ICD6 0.50 mm to (301.5, 265.5)
- moved ICE6 0.50 mm to (301.5, 245.0)
Other:
- outline, holes or cut-outs redrawn
Changed lines of the file:
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@@
     (property "ki_keywords" "connector")
     (attr through_hole)
-    (fp_text reference "LAMPENSPALTEN1" (at 0 -2.33 180) (layer "F.SilkS")
+    (fp_text reference "LAMPENSPALTEN1" (at 3.5 18.5 270) (layer "F.SilkS")
         (effects (font (size 1 1) (thickness 0.15)))
     )
@@
   )
   (footprint "Package_DIP:DIP-24_W15.24mm" (layer "F.Cu")
-    (at 307.06 286 90)
+    (at 306.56 286 90)
     (descr "24-lead though-hole mounted DIP package, row spacing 15.24 mm (600 mils)")
     (tags "THT DIP DIL PDIP 2.54mm 15.24mm 600mil")
@@
     (property "ki_keywords" "CMOS SWITCH")
     (attr through_hole)
-    (fp_text reference "ICG10-1" (at 2.5 12.2 180) (layer "B.SilkS")
+    (fp_text reference "ICG10-1" (at 3 11.7 180) (layer "B.SilkS")
         (effects (font (size 1 1) (thickness 0.15)) (justify mirror))
     )
@@
   )
   (footprint "Connector_PinHeader_2.54mm:PinHeader_1x20_P2.54mm_Vertical" (layer "F.Cu")
-    (at 442 178)
+    (at 442 170.46)
     (descr "Through hole straight pin header, 1x20, 2.54mm pitch, single row")
     (tags "Through hole pin header THT 1x20 2.54mm single row")
@@
     (property "ki_keywords" "connector")
     (attr through_hole)
-    (fp_text reference "SERVICEANZEIGE+TASTATUR1" (at 0 -2.33) (layer "F.SilkS")
+    (fp_text reference "SERVICEANZEIGE+TASTATUR1" (at 3.5 25 90) (layer "F.SilkS")
         (effects (font (size 1 1) (thickness 0.15)))
     )
@@
   )
   (footprint "Package_DIP:DIP-16_W7.62mm" (layer "F.Cu")
-    (at 241.76 187 90)
+    (at 244.3 187 90)
     (descr "16-lead though-hole mounted DIP package, row spacing 7.62 mm (300 mils)")
     (tags "THT DIP DIL PDIP 2.54mm 7.62mm 300mil")
@@
     (property "ki_keywords" "connector")
     (attr through_hole)
-    (fp_text reference "LEISTUNGSNETZ1" (at 0 -2.33) (layer "F.SilkS")
+    (fp_text reference "LEISTUNGSNETZ1" (at 3.5 9.5 90) (layer "F.SilkS")
         (effects (font (size 1 1) (thickness 0.15)))
     )
@@
   )
   (footprint "Package_DIP:DIP-28_W15.24mm" (layer "F.Cu")
-    (at 301.98 265.5 90)
+    (at 301.48 265.5 90)
     (descr "28-lead though-hole mounted DIP package, row spacing 15.24 mm (600 mils)")
     (tags "THT DIP DIL PDIP 2.54mm 15.24mm 600mil")
@@
     (property "ki_keywords" "R res resistor")
     (attr through_hole)
-    (fp_text reference "R40" (at 15.24 -4.32) (layer "F.SilkS")
+    (fp_text reference "R40" (at 38.245 0) (layer "F.SilkS")
         (effects (font (size 1 1) (thickness 0.15)))
     )
@@
     (property "ki_keywords" "connector")
     (attr through_hole)
-    (fp_text reference "SIGNALNETZ1" (at 0 -2.33) (layer "F.SilkS")
+    (fp_text reference "SIGNALNETZ1" (at 4 7 90) (layer "F.SilkS")
         (effects (font (size 1 1) (thickness 0.15)))
     )
@@
   )
   (footprint "Package_DIP:DIP-14_W7.62mm" (layer "F.Cu")
-    (at 414.26 174 90)
+    (at 414.26 175.3 90)
     (descr "14-lead though-hole mounted DIP package, row spacing 7.62 mm (300 mils)")
     (tags "THT DIP DIL PDIP 2.54mm 7.62mm 300mil")
@@
   )
   (footprint "Package_DIP:DIP-16_W7.62mm" (layer "F.Cu")
-    (at 412.42 206 90)
+    (at 411.8 206 90)
     (descr "16-lead though-hole mounted DIP package, row spacing 7.62 mm (300 mils)")
     (tags "THT DIP DIL PDIP 2.54mm 7.62mm 300mil")
@@
     (property "ki_keywords" "R network parallel topology isolated")
     (attr through_hole)
-    (fp_text reference "RM81" (at 3.81 -2.33 90) (layer "F.SilkS")
-        (effects (font (size 1 1) (thickness 0.15)))
+    (fp_text reference "RM81" (at 3.81 24.58 180) (layer "B.SilkS")
+        (effects (font (size 1 1) (thickness 0.15)) (justify mirror))
     )
     (fp_text value "R_Pack08" (at 3.81 20.11 90) (layer "F.Fab")
@@
   )
   (footprint "Package_DIP:DIP-28_W15.24mm" (layer "F.Cu")
-    (at 301.98 245 90)
+    (at 301.48 245 90)
     (descr "28-lead though-hole mounted DIP package, row spacing 15.24 mm (600 mils)")
     (tags "THT DIP DIL PDIP 2.54mm 15.24mm 600mil")
@@
     (property "ki_keywords" "connector")
     (attr through_hole)
-    (fp_text reference "EINGAENGE1" (at 0 -2.33 90) (layer "F.SilkS")
+    (fp_text reference "EINGAENGE1" (at 4.5 8.5 180) (layer "F.SilkS")
         (effects (font (size 1 1) (thickness 0.15)))
     )
@@
     )
   )
-  (gr_rect (start 305.5 269.5) (end 336.5 287)
+  (gr_rect (start 305 269.5) (end 336 287)
     (stroke (width 0.15) (type default)) (fill none) (layer "B.SilkS"))
-  (gr_rect (start 300.5 228.5) (end 336.5 246)
+  (gr_rect (start 300 228.5) (end 336 246)
     (stroke (width 0.15) (type default)) (fill none) (layer "B.SilkS"))
-  (gr_rect (start 300.5 249) (end 336.5 266.5)
+  (gr_rect (start 300 249) (end 336 266.5)
     (stroke (width 0.15) (type default)) (fill none) (layer "B.SilkS"))
   (gr_circle (center 354 335) (end 356.5 335)
@@
   (gr_line (start 140 340) (end 140 80)
     (stroke (width 0.2) (type solid)) (layer "Edge.Cuts"))
-  (gr_circle (center 301 335) (end 302.5 335)
+  (gr_circle (center 300 335) (end 301.5 335)
     (stroke (width 0.1) (type default)) (fill none) (layer "Edge.Cuts"))
   (gr_line (start 140 80) (end 450 80)
@@
   (gr_circle (center 298 85) (end 299.5 85)
     (stroke (width 0.1) (type default)) (fill none) (layer "Edge.Cuts"))
-  (gr_circle (center 292 335) (end 293.5 335)
+  (gr_circle (center 291 335) (end 292.5 335)
     (stroke (width 0.1) (type default)) (fill none) (layer "Edge.Cuts"))
   (gr_circle (center 289 85) (end 290.5 85)
     (stroke (width 0.1) (type default)) (fill none) (layer "Edge.Cuts"))
-  (gr_text "ICD6" (at 311 257.5) (layer "B.SilkS")
+  (gr_text "ICD6" (at 311.5 256) (layer "B.SilkS")
     (effects (font (size 1 1) (thickness 0.15)) (justify mirror))
   )
-  (gr_text "ICE6" (at 310.5 236) (layer "B.SilkS")
+  (gr_text "ICE6" (at 311.5 234.5) (layer "B.SilkS")
     (effects (font (size 1 1) (thickness 0.15)) (justify mirror))
   )
-  (gr_text "ICC6" (at 316 275) (layer "B.SilkS")
+  (gr_text "ICC6" (at 311.5 273.5) (layer "B.SilkS")
     (effects (font (size 1 1) (thickness 0.15)) (justify mirror))
   )
@@
   )
   (dimension (type aligned) (layer "User.1")
-    (pts (xy 292 335) (xy 301 335))
+    (pts (xy 291 335) (xy 300 335))
     (height 15)
-    (gr_text "9,0000 mm" (at 296.5 348.85) (layer "User.1")
+    (gr_text "9,0000 mm" (at 295.5 348.85) (layer "User.1")
       (effects (font (size 1 1) (thickness 0.15)))
     )
@@
     (polygon
       (pts
-        (xy 298.5 332.5)
-        (xy 303.5 332.5)
-        (xy 303.5 337)
-        (xy 298.5 337)
+        (xy 297.5 332.5)
+        (xy 302.5 332.5)
+        (xy 302.5 337)
+        (xy 297.5 337)
       )
     )
@@
     (polygon
       (pts
-        (xy 289.5 332.5)
-        (xy 294.5 332.5)
-        (xy 294.5 337)
-        (xy 289.5 337)
+        (xy 288.5 332.5)
+        (xy 293.5 332.5)
+        (xy 293.5 337)
+        (xy 288.5 337)
       )
     )
@@
       )
     )
+  )
+  (zone (net 7) (net_name "GND") (layer "F.Cu") (hatch edge 0.5)
+    (priority 1)
+    (connect_pads (clearance 0.508))
+    (min_thickness 0.25) (filled_areas_thickness no)
+    (fill (thermal_gap 0.5) (thermal_bridge_width 0.5))
+    (polygon
+      (pts
+        (xy 140 340)
+        (xy 450 340)
+        (xy 450 330.5)
+        (xy 140 330.5)
+      )
+    )

Commit message: mehr anschluss
Parts:
- added BATTERIE2: Battery_Cell, Battery:BatteryHolder_Keystone_2460_1xAA, F.Cu at (247.8, 319.0)
- added GONG1: Conn_01x02_Pin, Connector_PinHeader_2.54mm:PinHeader_1x02_P2.54mm_Vertical, F.Cu at (219.2, 88.0)
- added LAMPENZEILEN1: Conn_01x16_Pin, Connector_PinHeader_2.54mm:PinHeader_1x16_P2.54mm_Vertical, F.Cu at (148.0, 169.5)
- added LAUTSPRECHER1: Conn_01x06_Pin, Connector_PinHeader_2.54mm:PinHeader_1x06_P2.54mm_Vertical, F.Cu at (429.4, 90.0)
- added LEUCHTZIFFERNANZEIGE1: Conn_01x12_Pin, Connector_PinHeader_2.54mm:PinHeader_1x12_P2.54mm_Vertical, F.Cu at (157.9, 88.0)
- moved LAMPENSPALTEN1 6.60 mm to (148.0, 126.6)
- moved R2 0.56 mm to (177.5, 143.4)
- moved TR2 0.56 mm to (177.5, 117.1)
- moved ICC6 0.50 mm to (306.6, 285.5)
- moved ICD6 0.50 mm to (301.5, 265.0)
- moved ICE6 0.50 mm to (301.5, 244.5)
- moved R1 0.50 mm to (169.5, 143.2)
- moved R10 0.50 mm to (185.5, 143.4)
- moved R11 0.50 mm to (193.5, 143.4)
- moved TR1 0.50 mm to (169.4, 116.8)
- moved TR10 0.50 mm to (185.5, 117.1)
- moved TR11 0.50 mm to (193.5, 117.1)
- moved TR32 0.50 mm to (222.0, 163.0)

Commit message: rechts
Parts:
- added AUSWERFER+SPERRMAG1: Conn_01x06_Pin, Connector_PinHeader_2.54mm:PinHeader_1x06_P2.54mm_Vertical, F.Cu at (442.0, 127.4)
- added LEISTUNGSAUSGAENGE1: Conn_01x10_Pin, Connector_PinHeader_2.54mm:PinHeader_1x10_P2.54mm_Vertical, F.Cu at (401.3, 88.0)
- added MATRIX-EINGAENGE1: Conn_01x06_Pin, Connector_PinHeader_2.54mm:PinHeader_1x06_P2.54mm_Vertical, F.Cu at (442.0, 149.4)
- added MUENZANNAHME1: Conn_01x20_Pin, Connector_PinHeader_2.54mm:PinHeader_1x20_P2.54mm_Vertical, F.Cu at (442.5, 226.4)
- added SERIELLE_DATEN1: Conn_01x08_Pin, Connector_PinHeader_2.54mm:PinHeader_1x08_P2.54mm_Vertical, F.Cu at (442.0, 307.4)
- moved BATTERIE2 4.01 mm to (248.0, 315.0)
- moved LAUTSPRECHER1 2.13 mm to (430.1, 88.0)
- moved LAMPENSPALTEN1 0.99 mm to (147.5, 125.7)
- moved LAMPENZEILEN1 0.78 mm to (147.5, 170.1)
- moved R1 0.60 mm to (169.0, 143.5)
- moved TR1 0.55 mm to (168.9, 117.1)
- moved R10 0.50 mm to (185.0, 143.4)
- moved R11 0.50 mm to (193.0, 143.4)
- moved R12 0.50 mm to (200.5, 143.4)
- moved R13 0.50 mm to (207.5, 143.4)
- moved R2 0.50 mm to (177.0, 143.4)
- moved TR10 0.50 mm to (185.0, 117.1)
- moved TR11 0.50 mm to (193.0, 117.1)
- moved TR12 0.50 mm to (200.5, 117.1)
- moved TR13 0.50 mm to (207.5, 117.1)
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Routing:
- net Net-(TR1-E): track 49.1 -> 53.1 mm

Commit message: LED
Parts:
- added LED1: LED, LED_THT:LED_D3.0mm, F.Cu at (239.0, 114.0)
- added LED2: LED, LED_THT:LED_D3.0mm, F.Cu at (320.2, 131.5)
- added LED3: LED, LED_THT:LED_D3.0mm, F.Cu at (327.2, 131.5)
- added LED4: LED, LED_THT:LED_D3.0mm, F.Cu at (319.2, 300.0)
- added LED5: LED, LED_THT:LED_D3.0mm, F.Cu at (230.7, 294.0)
- added SW1: SW_DIP_x04, Button_Switch_THT:SW_DIP_SPSTx04_Slide_9.78x12.34mm_W7.62mm_P2.54mm, F.Cu at (211.6, 254.9)
- added TASTEN1: Conn_01x06_Pin, Connector_PinHeader_2.54mm:PinHeader_1x06_P2.54mm_Vertical, F.Cu at (148.0, 269.6)
- added TUERSCHALTER+SPIELZAEHLER1: Conn_01x04_Pin, Connector_PinHeader_2.54mm:PinHeader_1x04_P2.54mm_Vertical, F.Cu at (148.0, 315.7)
- added WALZENSTEUERUNG1: Conn_01x20_Pin, Connector_PinHeader_2.54mm:PinHeader_1x20_P2.54mm_Vertical, F.Cu at (147.5, 177.3)
- added ZUSATZTASTEN1: Conn_01x08_Pin, Connector_PinHeader_2.54mm:PinHeader_1x08_P2.54mm_Vertical, F.Cu at (148.0, 289.4)
- added ZUSATZWALZEN1: Conn_01x12_Pin, Connector_PinHeader_2.54mm:PinHeader_1x12_P2.54mm_Vertical, F.Cu at (148.0, 233.2)
- moved LEISTUNGSAUSGAENGE1 3.50 mm to (397.8, 88.0)
- moved BATTERIE2 3.00 mm to (248.0, 312.0)
- moved MATRIX-EINGAENGE1 2.00 mm to (442.0, 147.4)
- moved AUSWERFER+SPERRMAG1 1.46 mm to (442.0, 125.9)
- moved LEUCHTZIFFERNANZEIGE1 1.32 mm to (156.6, 88.0)
- moved SERIELLE_DATEN1 1.12 mm to (442.0, 308.5)
- moved MUENZANNAHME1 1.10 mm to (442.5, 227.5)

Commit message: spin
Parts:
- moved WALZENSTEUERUNG1 46.1 mm to (147.5, 223.4), turned to 180 degrees
- moved ZUSATZWALZEN1 26.9 mm to (148.0, 260.0), turned to 180 degrees
- moved ZUSATZTASTEN1 18.8 mm to (148.0, 308.1), turned to 180 degrees
- moved SW1 14.5 mm to (198.8, 261.7)
- moved TUERSCHALTER+SPIELZAEHLER1 11.2 mm to (148.0, 326.9), turned to 180 degrees
- moved TASTEN1 10.9 mm to (148.0, 280.6), turned to 180 degrees
- moved LED2 6.93 mm to (315.0, 136.0), turned to 90 degrees
- moved LED3 6.93 mm to (322.0, 136.0), turned to 90 degrees
- moved LED1 3.21 mm to (240.0, 117.0), turned to 90 degrees
- moved LED4 2.26 mm to (317.5, 301.5), turned to 180 degrees
- moved ICH4-1 1.00 mm to (245.3, 187.0)
- moved LAMPENSPALTEN1 0.66 mm to (147.5, 125.1)
Routing:
- net GND: track 0.00 -> 10.3 mm, vias 0 -> 3

Commit message: 3d fix
Parts:
- moved TASTEN1 4.92 mm to (148.0, 285.5)
- moved ZUSATZWALZEN1 2.96 mm to (148.0, 263.0)
- moved WALZENSTEUERUNG1 2.64 mm to (147.5, 226.0)
- moved TUERSCHALTER+SPIELZAEHLER1 2.50 mm to (148.0, 329.4)
- moved ZUSATZTASTEN1 2.00 mm to (148.0, 310.1)
Changed lines of the file:
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@@
   )
   (footprint "Connector_PinHeader_2.54mm:PinHeader_1x20_P2.54mm_Vertical" (layer "F.Cu")
-    (at 147.5 223.36 180)
+    (at 147.5 226 180)
     (descr "Through hole straight pin header, 1x20, 2.54mm pitch, single row")
     (tags "Through hole pin header THT 1x20 2.54mm single row")
@@
   )
   (footprint "Connector_PinHeader_2.54mm:PinHeader_1x04_P2.54mm_Vertical" (layer "F.Cu")
-    (at 148 326.86 180)
+    (at 148 329.36 180)
     (descr "Through hole straight pin header, 1x04, 2.54mm pitch, single row")
     (tags "Through hole pin header THT 1x04 2.54mm single row")
@@
   )
   (footprint "Connector_PinHeader_2.54mm:PinHeader_1x06_P2.54mm_Vertical" (layer "F.Cu")
-    (at 148 280.58 180)
+    (at 148 285.5 180)
     (descr "Through hole straight pin header, 1x06, 2.54mm pitch, single row")
     (tags "Through hole pin header THT 1x06 2.54mm single row")
@@
   )
   (footprint "Connector_PinHeader_2.54mm:PinHeader_1x08_P2.54mm_Vertical" (layer "F.Cu")
-    (at 148 308.13 180)
+    (at 148 310.13 180)
     (descr "Through hole straight pin header, 1x08, 2.54mm pitch, single row")
     (tags "Through hole pin header THT 1x08 2.54mm single row")
@@
   )
   (footprint "Connector_PinHeader_2.54mm:PinHeader_1x12_P2.54mm_Vertical" (layer "F.Cu")
-    (at 148 260.04 180)
+    (at 148 263 180)
     (descr "Through hole straight pin header, 1x12, 2.54mm pitch, single row")
     (tags "Through hole pin header THT 1x12 2.54mm single row")
@@
   (gr_rect (start 305 269) (end 336 286.5)
     (stroke (width 0.15) (type default)) (fill none) (layer "B.SilkS"))
-  (gr_rect (start 146.5 289) (end 149.5 309.5)
+  (gr_rect (start 440 168.5) (end 444 220.5)
     (stroke (width 0.15) (type default)) (fill none) (layer "B.SilkS"))
-  (gr_rect (start 146 85.5) (end 149 126.5)
+  (gr_rect (start 146 290) (end 150 312.5)
     (stroke (width 0.15) (type default)) (fill none) (layer "B.SilkS"))
-  (gr_rect (start 146 130.5) (end 149 171.5)
+  (gr_rect (start 145.5 85) (end 149.5 127)
+    (stroke (width 0.15) (type default)) (fill none) (layer "B.SilkS"))
+  (gr_rect (start 440 96) (end 444 117.5)
+    (stroke (width 0.15) (type default)) (fill none) (layer "B.SilkS"))
+  (gr_rect (start 440 306.5) (end 444 328)
+    (stroke (width 0.15) (type default)) (fill none) (layer "B.SilkS"))
+  (gr_rect (start 145.5 130) (end 149.5 172.5)
     (stroke (width 0.15) (type default)) (fill none) (layer "B.SilkS"))
   (gr_rect (start 300 228) (end 336 245.5)
     (stroke (width 0.15) (type default)) (fill none) (layer "B.SilkS"))
-  (gr_rect (start 146 173.5) (end 149 224.5)
+  (gr_rect (start 440 284) (end 444 300.5)
     (stroke (width 0.15) (type default)) (fill none) (layer "B.SilkS"))
-  (gr_rect (start 146.5 266.5) (end 149.5 282)
+  (gr_rect (start 145.5 175.5) (end 149.5 228)
     (stroke (width 0.15) (type default)) (fill none) (layer "B.SilkS"))
-  (gr_rect (start 146.5 230.5) (end 149.5 261.5)
+  (gr_rect (start 146 270.5) (end 150 287.5)
+    (stroke (width 0.15) (type default)) (fill none) (layer "B.SilkS"))
+  (gr_rect (start 146 233) (end 150 265)
     (stroke (width 0.15) (type default)) (fill none) (layer "B.SilkS"))
   (gr_rect (start 190 260.5) (end 200 270.5)
@@
   (gr_rect (start 300 248.5) (end 336 266)
     (stroke (width 0.15) (type default)) (fill none) (layer "B.SilkS"))
-  (gr_rect (start 146.5 318) (end 149.5 328)
+  (gr_rect (start 396 86) (end 422.5 90)
+    (stroke (width 0.15) (type default)) (fill none) (layer "B.SilkS"))
+  (gr_rect (start 440 124) (end 444 140.5)
+    (stroke (width 0.15) (type default)) (fill none) (layer "B.SilkS"))
+  (gr_rect (start 440.5 225.5) (end 444.5 277.5)
+    (stroke (width 0.15) (type default)) (fill none) (layer "B.SilkS"))
+  (gr_rect (start 440 145.5) (end 444 162)
+    (stroke (width 0.15) (type default)) (fill none) (layer "B.SilkS"))
+  (gr_rect (start 146 319.5) (end 150 331.5)
+    (stroke (width 0.15) (type default)) (fill none) (layer "B.SilkS"))
+  (gr_rect (start 428.5 86) (end 444.5 90)
     (stroke (width 0.15) (type default)) (fill none) (layer "B.SilkS"))
   (gr_circle (center 354 335) (end 356.5 335)
@@
     (connect_pads (clearance 0.508))
     (min_thickness 0.25) (filled_areas_thickness no)
-    (fill (thermal_gap 0.5) (thermal_bridge_width 0.5))
+    (fill yes (thermal_gap 0.5) (thermal_bridge_width 0.5))
     (polygon
       (pts
@@
     (connect_pads (clearance 0.508))
     (min_thickness 0.25) (filled_areas_thickness no)
-    (fill (thermal_gap 0.5) (thermal_bridge_width 0.5))
+    (fill yes (thermal_gap 0.5) (thermal_bridge_width 0.5))
     (polygon
       (pts
