File: weisse_cpu.kicad_pcb (KiCad board)
At the start: 2 copper layers, 310 x 260 mm, 51 parts, among them SW1 SW_DIP_x04

Commit message: 3d zoom
Parts:
- moved LED2 10.9 mm to (305.0, 140.5)
- moved LED3 10.9 mm to (312.0, 140.5)
- moved LED5 9.58 mm to (229.5, 303.5)
- moved SW1 8.39 mm to (190.6, 259.9)
- moved LED1 2.13 mm to (238.0, 117.8)
- moved LED4 2.06 mm to (315.5, 302.0)
- moved ZUSATZTASTEN1 1.87 mm to (148.0, 312.0)
- moved ZUSATZWALZEN1 0.94 mm to (148.0, 263.9)
- moved WALZENSTEUERUNG1 0.64 mm to (148.0, 226.4)
- moved LAMPENZEILEN1 0.50 mm to (147.5, 170.6)
- moved SERIELLE_DATEN1 0.50 mm to (442.5, 308.5)
- moved SIGNALNETZ1 0.50 mm to (442.5, 286.0)
Routing:
- net GND: vias 3 -> 2
- added copper zone on B.Cu, net GND
Changed lines of the file:
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@@
   )
   (footprint "Connector_PinHeader_2.54mm:PinHeader_1x20_P2.54mm_Vertical" (layer "F.Cu")
-    (at 147.5 226 180)
+    (at 148 226.4 180)
     (descr "Through hole straight pin header, 1x20, 2.54mm pitch, single row")
     (tags "Through hole pin header THT 1x20 2.54mm single row")
@@
   )
   (footprint "LED_THT:LED_D3.0mm" (layer "F.Cu")
-    (at 317.54 301.5 180)
+    (at 315.54 302 180)
     (descr "LED, diameter 3.0mm, 2 pins")
     (tags "LED diameter 3.0mm 2 pins")
@@
     (property "ki_keywords" "connector")
     (attr through_hole)
-    (fp_text reference "TUERSCHALTER+SPIELZAEHLER1" (at 3.5 4.36 90) (layer "F.SilkS")
+    (fp_text reference "TUERSCHALTER+SPIELZAEHLER1" (at 3.5 2.49 90) (layer "F.SilkS")
         (effects (font (size 1 1) (thickness 0.15)))
     )
@@
   )
   (footprint "LED_THT:LED_D3.0mm" (layer "F.Cu")
-    (at 314.96 136 90)
+    (at 305 140.5 90)
     (descr "LED, diameter 3.0mm, 2 pins")
     (tags "LED diameter 3.0mm 2 pins")
@@
   )
   (footprint "LED_THT:LED_D3.0mm" (layer "F.Cu")
-    (at 240 117.04 90)
+    (at 238 117.775 90)
     (descr "LED, diameter 3.0mm, 2 pins")
     (tags "LED diameter 3.0mm 2 pins")
@@
   )
   (footprint "LED_THT:LED_D3.0mm" (layer "F.Cu")
-    (at 321.96 136 90)
+    (at 312 140.5 90)
     (descr "LED, diameter 3.0mm, 2 pins")
     (tags "LED diameter 3.0mm 2 pins")
@@
   )
   (footprint "Connector_PinHeader_2.54mm:PinHeader_1x08_P2.54mm_Vertical" (layer "F.Cu")
-    (at 442 308.5)
+    (at 442.5 308.5)
     (descr "Through hole straight pin header, 1x08, 2.54mm pitch, single row")
     (tags "Through hole pin header THT 1x08 2.54mm single row")
@@
   )
   (footprint "Button_Switch_THT:SW_DIP_SPSTx04_Slide_9.78x12.34mm_W7.62mm_P2.54mm" (layer "F.Cu")
-    (at 198.8 261.7325 -90)
+    (at 190.62 259.88 -90)
     (descr "4x-dip-switch SPST , Slide, row spacing 7.62 mm (300 mils), body size 9.78x12.34mm (see e.g. https://www.ctscorp.com/wp-content/uploads/206-208.pdf)")
     (tags "DIP Switch SPST Slide 7.62mm 300mil")
@@
   )
   (footprint "Connector_PinHeader_2.54mm:PinHeader_1x16_P2.54mm_Vertical" (layer "F.Cu")
-    (at 147.5 170.1 180)
+    (at 147.5 170.6 180)
     (descr "Through hole straight pin header, 1x16, 2.54mm pitch, single row")
     (tags "Through hole pin header THT 1x16 2.54mm single row")
@@
   )
   (footprint "LED_THT:LED_D3.0mm" (layer "F.Cu")
-    (at 230.725 294)
+    (at 229.46 303.5)
     (descr "LED, diameter 3.0mm, 2 pins")
     (tags "LED diameter 3.0mm 2 pins")
@@
   )
   (footprint "Connector_PinHeader_2.54mm:PinHeader_1x06_P2.54mm_Vertical" (layer "F.Cu")
-    (at 442 286)
+    (at 442.5 286)
     (descr "Through hole straight pin header, 1x06, 2.54mm pitch, single row")
     (tags "Through hole pin header THT 1x06 2.54mm single row")
@@
   )
   (footprint "Connector_PinHeader_2.54mm:PinHeader_1x08_P2.54mm_Vertical" (layer "F.Cu")
-    (at 148 310.13 180)
+    (at 148 312 180)
     (descr "Through hole straight pin header, 1x08, 2.54mm pitch, single row")
     (tags "Through hole pin header THT 1x08 2.54mm single row")
@@
   )
   (footprint "Connector_PinHeader_2.54mm:PinHeader_1x12_P2.54mm_Vertical" (layer "F.Cu")
-    (at 148 263 180)
+    (at 148 263.94 180)
     (descr "Through hole straight pin header, 1x12, 2.54mm pitch, single row")
     (tags "Through hole pin header THT 1x12 2.54mm single row")
@@
   (gr_rect (start 305 269) (end 336 286.5)
     (stroke (width 0.15) (type default)) (fill none) (layer "B.SilkS"))
-  (gr_rect (start 440 168.5) (end 444 220.5)
+  (gr_rect (start 440 168.5) (end 444.5 220.5)
     (stroke (width 0.15) (type default)) (fill none) (layer "B.SilkS"))
-  (gr_rect (start 146 290) (end 150 312.5)
+  (gr_rect (start 146 291.87) (end 150 314.37)
     (stroke (width 0.15) (type default)) (fill none) (layer "B.SilkS"))
-  (gr_rect (start 145.5 85) (end 149.5 127)
+  (gr_rect (start 145.5 85) (end 150 127)
     (stroke (width 0.15) (type default)) (fill none) (layer "B.SilkS"))
-  (gr_rect (start 440 96) (end 444 117.5)
+  (gr_rect (start 440 96) (end 444.5 118)
     (stroke (width 0.15) (type default)) (fill none) (layer "B.SilkS"))
-  (gr_rect (start 440 306.5) (end 444 328)
+  (gr_rect (start 440.5 306.5) (end 445 328)
     (stroke (width 0.15) (type default)) (fill none) (layer "B.SilkS"))
-  (gr_rect (start 145.5 130) (end 149.5 172.5)
+  (gr_rect (start 145 130.5) (end 150 173)
     (stroke (width 0.15) (type default)) (fill none) (layer "B.SilkS"))
   (gr_rect (start 300 228) (end 336 245.5)
     (stroke (width 0.15) (type default)) (fill none) (layer "B.SilkS"))
-  (gr_rect (start 440 284) (end 444 300.5)
+  (gr_rect (start 440.5 284) (end 445 300.5)
     (stroke (width 0.15) (type default)) (fill none) (layer "B.SilkS"))
-  (gr_rect (start 145.5 175.5) (end 149.5 228)
+  (gr_rect (start 145.5 175.9) (end 150 228.4)
     (stroke (width 0.15) (type default)) (fill none) (layer "B.SilkS"))
-  (gr_rect (start 146 270.5) (end 150 287.5)
+  (gr_rect (start 145.5 270.5) (end 150 288)
     (stroke (width 0.15) (type default)) (fill none) (layer "B.SilkS"))
-  (gr_rect (start 146 233) (end 150 265)
+  (gr_rect (start 145.5 233.94) (end 150 265.94)
     (stroke (width 0.15) (type default)) (fill none) (layer "B.SilkS"))
-  (gr_rect (start 190 260.5) (end 200 270.5)
+  (gr_rect (start 181.82 258.6475) (end 191.82 268.6475)
     (stroke (width 0.15) (type default)) (fill none) (layer "B.SilkS"))
   (gr_rect (start 300 248.5) (end 336 266)
     (stroke (width 0.15) (type default)) (fill none) (layer "B.SilkS"))
-  (gr_rect (start 396 86) (end 422.5 90)
+  (gr_rect (start 396 85.5) (end 422.5 90)
     (stroke (width 0.15) (type default)) (fill none) (layer "B.SilkS"))
-  (gr_rect (start 440 124) (end 444 140.5)
+  (gr_rect (start 440 124) (end 444.5 140.5)
     (stroke (width 0.15) (type default)) (fill none) (layer "B.SilkS"))
-  (gr_rect (start 440.5 225.5) (end 444.5 277.5)
+  (gr_rect (start 440.5 225.5) (end 445 277.5)
     (stroke (width 0.15) (type default)) (fill none) (layer "B.SilkS"))
-  (gr_rect (start 440 145.5) (end 444 162)
+  (gr_rect (start 440 145.5) (end 444.5 162.5)
     (stroke (width 0.15) (type default)) (fill none) (layer "B.SilkS"))
-  (gr_rect (start 146 319.5) (end 150 331.5)
+  (gr_rect (start 145.5 319) (end 150.5 331.5)
     (stroke (width 0.15) (type default)) (fill none) (layer "B.SilkS"))
-  (gr_rect (start 428.5 86) (end 444.5 90)
+  (gr_rect (start 428.5 85.5) (end 445 90)
     (stroke (width 0.15) (type default)) (fill none) (layer "B.SilkS"))
   (gr_circle (center 354 335) (end 356.5 335)
@@
   (segment (start 209 84) (end 209 83) (width 1) (layer "F.Cu") (net 7))
   (via (at 208.5 84.5) (size 0.8) (drill 0.4) (layers "F.Cu" "B.Cu") (net 7))
-  (via (at 437 170.5) (size 0.8) (drill 0.4) (layers "F.Cu" "B.Cu") (net 7))
-  (via (at 437 170.5) (size 0.8) (drill 0.4) (layers "F.Cu" "B.Cu") (net 7))
+  (via (at 437.48 170.5) (size 0.8) (drill 0.4) (layers "F.Cu" "B.Cu") (net 7))
   (segment (start 208.24 88) (end 208.24 84.76) (width 1) (layer "B.Cu") (net 7))
   (segment (start 208.24 84.76) (end 208.5 84.5) (width 1) (layer "B.Cu") (net 7))
-  (segment (start 437.04 170.46) (end 437 170.5) (width 1) (layer "B.Cu") (net 7))
-  (segment (start 442 170.46) (end 437.04 170.46) (width 1) (layer "B.Cu") (net 7))
+  (segment (start 442.48 170.46) (end 437.52 170.46) (width 1) (layer "B.Cu") (net 7))
   (segment (start 169 123.18) (end 169 117.235) (width 1) (layer "F.Cu") (net 144))
   (segment (start 169 117.235) (end 168.945 117.18) (width 1) (layer "F.Cu") (net 144))
@@
       )
     )
+  )
+  (zone (net 7) (net_name "GND") (layer "B.Cu") (hatch edge 0.5)
+    (priority 2)
+    (connect_pads (clearance 0.508))
+    (min_thickness 0.25) (filled_areas_thickness no)
+    (fill (thermal_gap 0.5) (thermal_bridge_width 0.5))
+    (polygon
+      (pts
+        (xy 140 80)
+        (xy 140 83.5)
+        (xy 151.5 83.5)
+        (xy 154.5 85)
+        (xy 450 85)
+        (xy 450 80)
+      )
+    )
