File: weisse_cpu.kicad_pcb (KiCad board)
At the start: 2 copper layers, 310 x 260 mm, 78 parts, among them SW1 SW_DIP_x04

Commit message: suqiggly lines
Routing:
- net Net-(LAMPENZEILEN1-Pin_1): track 2.54 -> 84.0 mm
- net Net-(LAMPENZEILEN1-Pin_3): track 2.54 -> 80.3 mm, vias 0 -> 1
- net Net-(LAMPENZEILEN1-Pin_5): track 2.54 -> 70.2 mm, vias 0 -> 2
- net Net-(LAMPENSPALTEN1-Pin_3): track 2.54 -> 68.1 mm, vias 0 -> 1
- net unconnected-(AUSWERFER+SPERRMAG1-Pin_5-Pad5): track 0.00 -> 63.5 mm, vias 0 -> 1
- net unconnected-(AUSWERFER+SPERRMAG1-Pin_4-Pad4): track 0.00 -> 61.6 mm, vias 0 -> 1
- net unconnected-(AUSWERFER+SPERRMAG1-Pin_3-Pad3): track 0.00 -> 58.6 mm, vias 0 -> 1
- net Net-(LAMPENSPALTEN1-Pin_5): track 2.54 -> 61.1 mm, vias 0 -> 1
- net unconnected-(AUSWERFER+SPERRMAG1-Pin_6-Pad6): track 0.00 -> 55.6 mm, vias 0 -> 1
- net Net-(LAMPENZEILEN1-Pin_7): track 2.54 -> 57.4 mm, vias 0 -> 1
- net unconnected-(AUSWERFER+SPERRMAG1-Pin_2-Pad2): track 0.00 -> 50.3 mm, vias 0 -> 1
- net Net-(LAMPENSPALTEN1-Pin_7): track 2.54 -> 52.4 mm, vias 0 -> 1
- net Net-(LAMPENZEILEN1-Pin_10): track 2.54 -> 48.2 mm, vias 0 -> 1
- net Net-(LAMPENSPALTEN1-Pin_10): track 2.54 -> 44.7 mm, vias 0 -> 1
- net +24V: track 0.00 -> 39.6 mm, vias 0 -> 2
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
Commit message: muenzen
Parts:
- added RM10: R_Pack08, Package_DIP:DIP-16_W7.62mm, F.Cu at (188.5, 178.5)
- added RM4: R_Pack08, Package_DIP:DIP-16_W7.62mm, F.Cu at (160.8, 250.0)
- added RM8: R_Pack08, Package_DIP:DIP-16_W7.62mm, F.Cu at (161.3, 318.0)
- added RM83: R_Pack08, Package_DIP:DIP-16_W7.62mm, F.Cu at (411.0, 236.5)
- added RM85: R_Pack08, Package_DIP:DIP-16_W7.62mm, F.Cu at (411.0, 267.0)
- renumbered RN1 to RM6
Connections:
- MUENZANNAHME1 pad 10: unconnected-(MUENZANNAHME1-Pin_10-Pad10) -> Net-(MUENZANNAHME1-Pin_10)
- MUENZANNAHME1 pad 11: unconnected-(MUENZANNAHME1-Pin_11-Pad11) -> Net-(MUENZANNAHME1-Pin_11)
- MUENZANNAHME1 pad 12: unconnected-(MUENZANNAHME1-Pin_12-Pad12) -> Net-(MUENZANNAHME1-Pin_12)
- MUENZANNAHME1 pad 13: unconnected-(MUENZANNAHME1-Pin_13-Pad13) -> Net-(MUENZANNAHME1-Pin_13)
- MUENZANNAHME1 pad 14: unconnected-(MUENZANNAHME1-Pin_14-Pad14) -> Net-(MUENZANNAHME1-Pin_14)
- MUENZANNAHME1 pad 15: unconnected-(MUENZANNAHME1-Pin_15-Pad15) -> Net-(MUENZANNAHME1-Pin_15)
- MUENZANNAHME1 pad 16: unconnected-(MUENZANNAHME1-Pin_16-Pad16) -> Net-(MUENZANNAHME1-Pin_16)
- MUENZANNAHME1 pad 17: unconnected-(MUENZANNAHME1-Pin_17-Pad17) -> Net-(MUENZANNAHME1-Pin_17)
- MUENZANNAHME1 pad 18: unconnected-(MUENZANNAHME1-Pin_18-Pad18) -> Net-(MUENZANNAHME1-Pin_18)
- MUENZANNAHME1 pad 6: unconnected-(MUENZANNAHME1-Pin_6-Pad6) -> Net-(MUENZANNAHME1-Pin_6)
- MUENZANNAHME1 pad 7: unconnected-(MUENZANNAHME1-Pin_7-Pad7) -> Net-(MUENZANNAHME1-Pin_7)
- MUENZANNAHME1 pad 8: unconnected-(MUENZANNAHME1-Pin_8-Pad8) -> Net-(MUENZANNAHME1-Pin_8)
- MUENZANNAHME1 pad 9: unconnected-(MUENZANNAHME1-Pin_9-Pad9) -> Net-(MUENZANNAHME1-Pin_9)
- WALZENANSTEUERUNG1 pad 2: unconnected-(WALZENANSTEUERUNG1-Pin_2-Pad2) -> Net-(RM4-R3.2)
- WALZENANSTEUERUNG1 pad 3: unconnected-(WALZENANSTEUERUNG1-Pin_3-Pad3) -> Net-(RM4-R4.2)
- WALZENANSTEUERUNG1 pad 4: unconnected-(WALZENANSTEUERUNG1-Pin_4-Pad4) -> Net-(RM4-R5.2)
- ZUSATZTASTEN1 pad 5: unconnected-(ZUSATZTASTEN1-Pin_5-Pad5) -> Net-(RM8-R7.2)
- ZUSATZTASTEN1 pad 6: unconnected-(ZUSATZTASTEN1-Pin_6-Pad6) -> Net-(RM8-R3.2)
Routing:
- net Net-(MUENZANNAHME1-Pin_13): track 0.00 -> 42.6 mm
- net Net-(MUENZANNAHME1-Pin_12): track 0.00 -> 38.3 mm
- net Net-(MUENZANNAHME1-Pin_11): track 0.00 -> 34.7 mm
- net Net-(RM8-R7.2): track 0.00 -> 33.0 mm
- net Net-(MUENZANNAHME1-Pin_10): track 0.00 -> 31.3 mm
- net Net-(RM6-R5.1): track 0.00 -> 28.6 mm
- net Net-(MUENZANNAHME1-Pin_9): track 0.00 -> 27.7 mm
- net Net-(MUENZANNAHME1-Pin_14): track 0.00 -> 26.6 mm
- net Net-(RM6-R4.1): track 0.00 -> 25.0 mm
- net Net-(RM8-R3.2): track 0.00 -> 23.9 mm
- net Net-(MUENZANNAHME1-Pin_15): track 0.00 -> 23.3 mm
- net Net-(MUENZANNAHME1-Pin_8): track 0.00 -> 23.1 mm
- net unconnected-(ZUSATZTASTEN1-Pin_4-Pad4): track 0.00 -> 21.6 mm, vias 0 -> 1
- net Net-(RM6-R3.1): track 0.00 -> 21.4 mm
- net Net-(MUENZANNAHME1-Pin_16): track 0.00 -> 20.3 mm
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
Commit message: logic
Parts:
- added ICB4: 74LS245, Package_DIP:DIP-20_W7.62mm, F.Cu at (240.5, 298.0)
- added ICC3: 74LS04, Package_DIP:DIP-14_W7.62mm, F.Cu at (220.0, 278.0)
- added ICD3: 74LS257, Package_DIP:DIP-16_W7.62mm, F.Cu at (217.6, 267.4)
- added Q1: Crystal, Crystal:Crystal_AT310_D3.0mm_L10.0mm_Vertical, F.Cu at (159.8, 265.8)
- added Q2: Crystal, Crystal:Crystal_HC18-U_Vertical, F.Cu at (209.5, 272.0)

Commit message: cpu
Parts:
- added ICB2: 8085, Package_DIP:DIP-40_W15.24mm, F.Cu at (186.9, 298.0)

Commit message: rtx 4060
Parts:
- added C159: C, Capacitor_THT:C_Rect_L9.0mm_W2.5mm_P7.50mm_MKT, F.Cu at (416.1, 274.8)
- added C160: C, Capacitor_THT:C_Rect_L9.0mm_W2.5mm_P7.50mm_MKT, F.Cu at (416.1, 282.6)
- added C161: C, Capacitor_THT:C_Rect_L9.0mm_W2.5mm_P7.50mm_MKT, F.Cu at (416.3, 290.2)
- added ICB10: 4066, Package_DIP:DIP-14_W7.62mm, F.Cu at (390.4, 297.8)
- added ICB9: 4066, Package_DIP:DIP-14_W7.62mm, F.Cu at (370.4, 297.8)
- added ICC10: 4066, Package_DIP:DIP-14_W7.62mm, F.Cu at (390.4, 282.4)
- added ICD10: 4066, Package_DIP:DIP-14_W7.62mm, F.Cu at (390.2, 267.2)
- added ICE10: 4066, Package_DIP:DIP-14_W7.62mm, F.Cu at (390.2, 251.8)
- added ICF10: 4066, Package_DIP:DIP-14_W7.62mm, F.Cu at (390.0, 236.8)

Commit message: transistoren
Parts:
- added ICB5: 74LS373, Package_DIP:DIP-20_W7.62mm, F.Cu at (271.1, 297.8)
- added ICD8: CD4051B, Package_DIP:DIP-16_W7.62mm, F.Cu at (342.5, 266.6)
- added ICF8: CD4051B, Package_DIP:DIP-16_W7.62mm, F.Cu at (342.2, 236.8)
- added TR70: Q_NPN_Darlington_BCE, Package_TO_SOT_THT:TO-220-3_Vertical, F.Cu at (340.6, 124.2)
- added TR71: Q_NPN_Darlington_BCE, Package_TO_SOT_THT:TO-220-3_Vertical, F.Cu at (347.0, 124.4)
- added TR72: Q_NPN_Darlington_BCE, Package_TO_SOT_THT:TO-220-3_Vertical, F.Cu at (353.4, 124.2)
- added TR73: Q_NPN_Darlington_BCE, Package_TO_SOT_THT:TO-220-3_Vertical, F.Cu at (359.6, 124.0)
- added TR80: Q_NPN_Darlington_BCE, Package_TO_SOT_THT:TO-220-3_Vertical, F.Cu at (366.0, 124.0)
- added TR81: Q_NPN_Darlington_BCE, Package_TO_SOT_THT:TO-220-3_Vertical, F.Cu at (372.4, 124.2)
- added TR82: Q_NPN_Darlington_BCE, Package_TO_SOT_THT:TO-220-3_Vertical, F.Cu at (378.6, 124.0)
- added TR83: Q_NPN_Darlington_BCE, Package_TO_SOT_THT:TO-220-3_Vertical, F.Cu at (385.2, 124.2)
- added TR95: Q_NPN_Darlington_BCE, Package_TO_SOT_THT:TO-220-3_Vertical, F.Cu at (391.4, 124.0)
- added TR96: Q_NPN_Darlington_BCE, Package_TO_SOT_THT:TO-220-3_Vertical, F.Cu at (398.0, 124.0)
- added TR97: Q_NPN_Darlington_BCE, Package_TO_SOT_THT:TO-220-3_Vertical, F.Cu at (404.2, 124.1)
Connections:
- ICB4 pad 10: unconnected-(ICB4-GND-Pad10) -> GND
- ICC3 pad 7: unconnected-(ICC3G-GND-Pad7) -> GND
- ICD3 pad 8: unconnected-(ICD3-GND-Pad8) -> GND
- ICH1 pad 8: unconnected-(ICH1C-VSS-Pad8) -> GND
Routing:
- net Net-(RM81-R1.1): track 0.00 -> 35.5 mm
- net Net-(TR70-E): track 0.00 -> 31.8 mm
- net (no net): track 0.00 -> 29.6 mm
- net Net-(TR82-E): track 0.00 -> 19.4 mm

Commit message: caps
Parts:
- added C20: C, Capacitor_THT:C_Rect_L7.0mm_W2.0mm_P5.00mm, F.Cu at (161.4, 300.4)
- added C21: C, Capacitor_THT:C_Rect_L7.0mm_W2.0mm_P5.00mm, F.Cu at (164.0, 300.4)
- added C22: C, Capacitor_THT:C_Rect_L7.0mm_W2.0mm_P5.00mm, F.Cu at (166.6, 300.4)
- added C23: C, Capacitor_THT:C_Rect_L7.0mm_W2.0mm_P5.00mm, F.Cu at (169.2, 300.4)
- added C24: C, Capacitor_THT:C_Rect_L7.0mm_W2.0mm_P5.00mm, F.Cu at (171.8, 300.4)
- added C25: C, Capacitor_THT:C_Rect_L7.0mm_W2.0mm_P5.00mm, F.Cu at (174.4, 300.4)
- added C26: C, Capacitor_THT:C_Rect_L7.0mm_W2.0mm_P5.00mm, F.Cu at (177.0, 300.4)
- added C27: C, Capacitor_THT:C_Rect_L7.0mm_W2.0mm_P5.00mm, F.Cu at (179.6, 300.4)
- added ICA7: 4066, Package_DIP:DIP-14_W7.62mm, F.Cu at (335.7, 315.4)
- added ICE2: 8256, Package_DIP:DIP-40_W15.24mm, F.Cu at (187.4, 252.4)
- added ICF3: 4028, Package_DIP:DIP-16_W7.62mm, F.Cu at (218.0, 227.2)
- added R29: R, Resistor_THT:R_Axial_DIN0414_L11.9mm_D4.5mm_P20.32mm_Horizontal, F.Cu at (229.8, 143.2)
- renumbered R29 to R28

Commit message: chips
Parts:
- added ICG10-2: 4066, Package_DIP:DIP-14_W7.62mm, F.Cu at (391.0, 221.8)
- added ICG8-1: 74LS290, Package_DIP:DIP-14_W7.62mm, F.Cu at (345.0, 206.6)
- added ICG8-2: 4040, Package_DIP:DIP-16_W7.62mm, F.Cu at (342.1, 221.6)
- added ICH10: 4066, Package_DIP:DIP-14_W7.62mm, F.Cu at (391.0, 191.2)
- added ICL10: NE556, Package_DIP:DIP-14_W7.62mm, F.Cu at (390.9, 160.6)
- added ICL8: 4013, Package_DIP:DIP-14_W7.62mm, F.Cu at (341.9, 156.2)
- added ICL9: 4093, Package_DIP:DIP-14_W7.62mm, F.Cu at (370.1, 156.4)
Routing:
- net Net-(RM4-R5.2): track 0.00 -> 42.2 mm
- net Net-(RM4-R4.2): track 0.00 -> 37.7 mm
- net Net-(RM4-R3.2): track 0.00 -> 33.1 mm
- net unconnected-(WALZENANSTEUERUNG1-Pin_5-Pad5): track 0.00 -> 31.8 mm, vias 0 -> 2
- net unconnected-(TASTEN1-Pin_5-Pad5): track 0.00 -> 28.9 mm, vias 0 -> 1
- net unconnected-(ZUSATZWALZEN1-Pin_1-Pad1): track 0.00 -> 6.54 mm, vias 0 -> 1
