File: weisse_cpu.kicad_sch (KiCad schematic)
At the start: 40 parts

Commit message: LED
Parts:
- added LED1, LED2, LED3, LED4, LED5: LED, LED_THT:LED_D3.0mm, symbol Device:LED
- added SW1: SW_DIP_x04, Button_Switch_THT:SW_DIP_SPSTx04_Slide_9.78x12.34mm_W7.62mm_P2.54mm, symbol Switch:SW_DIP_x04
- added TASTEN1: Conn_01x06_Pin, Connector_PinHeader_2.54mm:PinHeader_1x06_P2.54mm_Vertical, symbol Connector:Conn_01x06_Pin
- added TUERSCHALTER+SPIELZAEHLER1: Conn_01x04_Pin, Connector_PinHeader_2.54mm:PinHeader_1x04_P2.54mm_Vertical, symbol Connector:Conn_01x04_Pin
- added WALZENSTEUERUNG1: Conn_01x20_Pin, Connector_PinHeader_2.54mm:PinHeader_1x20_P2.54mm_Vertical, symbol Connector:Conn_01x20_Pin
- added ZUSATZTASTEN1: Conn_01x08_Pin, Connector_PinHeader_2.54mm:PinHeader_1x08_P2.54mm_Vertical, symbol Connector:Conn_01x08_Pin
- added ZUSATZWALZEN1: Conn_01x12_Pin, Connector_PinHeader_2.54mm:PinHeader_1x12_P2.54mm_Vertical, symbol Connector:Conn_01x12_Pin

Commit message: spin
Parts:
- renumbered WALZENSTEUERUNG1 to WALZENANSTEUERUNG1
Connections:
- net GND: now also WALZENANSTEUERUNG1.1 (Pin_1)
Changed lines of the file:
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@@
+    (stroke (width 0) (type default))
+  )
+  (wire (pts (xy 349.25 111.76) (xy 358.14 111.76))
     (stroke (width 0) (type default))
   )
@@
   (symbol (lib_id "Connector:Conn_01x20_Pin") (at 344.17 134.62 0) (unit 1)
     (in_bom yes) (on_board yes) (dnp no) (fields_autoplaced)
-    (property "Reference" "WALZENSTEUERUNG1" (at 344.805 106.68 0)
+    (property "Reference" "WALZENANSTEUERUNG1" (at 344.805 106.68 0)
       (effects (font (size 1.27 1.27)))
     )
@@
       (project "weisse_cpu"
         (path "/e63e39d7-6ac0-4ffd-8aa3-1841a4541b55"
-          (reference "WALZENSTEUERUNG1") (unit 1)
+          (reference "WALZENANSTEUERUNG1") (unit 1)
         )
       )
@@
         )
       )
+    )
+  )
+  (symbol (lib_name "GND_1") (lib_id "power:GND") (at 358.14 111.76 180) (unit 1)
+    (in_bom yes) (on_board yes) (dnp no) (fields_autoplaced)
+    (property "Reference" "#PWR01" (at 358.14 105.41 0)
+      (effects (font (size 1.27 1.27)) hide)
+    )
+    (property "Value" "GND" (at 358.14 106.68 0)
+      (effects (font (size 1.27 1.27)))
+    )
+    (property "Footprint" "" (at 358.14 111.76 0)
+      (effects (font (size 1.27 1.27)) hide)
+    )
+    (property "Datasheet" "" (at 358.14 111.76 0)
+      (effects (font (size 1.27 1.27)) hide)
+    )
+    (pin "1")
+    (instances
+      (project "weisse_cpu"
+        (path "/e63e39d7-6ac0-4ffd-8aa3-1841a4541b55"
+          (reference "#PWR01") (unit 1)
+        )
+      )

Commit message: resist
Parts:
- added R100, R90: R, Resistor_THT:R_Axial_Power_L25.0mm_W9.0mm_P30.48mm, symbol Device:R
Connections:
- net GND: now also LEISTUNGSAUSGAENGE1.2 (Pin_2)
- new net: R100.1, R90.2
Changed lines of the file:
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@@
+    (stroke (width 0) (type default))
+  )
+  (wire (pts (xy 241.3 201.93) (xy 247.65 201.93))
     (stroke (width 0) (type default))
   )
@@
   )
   (wire (pts (xy 45.72 166.37) (xy 55.88 166.37))
+    (stroke (width 0) (type default))
+  )
+  (wire (pts (xy 346.71 31.75) (xy 355.6 31.75))
     (stroke (width 0) (type default))
   )
@@
     )
   )
+  (symbol (lib_id "Device:R") (at 237.49 201.93 90) (unit 1)
+    (in_bom yes) (on_board yes) (dnp no) (fields_autoplaced)
+    (property "Reference" "R90" (at 237.49 195.58 90)
+      (effects (font (size 1.27 1.27)))
+    )
+    (property "Value" "R" (at 237.49 198.12 90)
+      (effects (font (size 1.27 1.27)))
+    )
+    (property "Footprint" "Resistor_THT:R_Axial_Power_L25.0mm_W9.0mm_P30.48mm" (at 237.49 203.708 90)
+      (effects (font (size 1.27 1.27)) hide)
+    )
+    (property "Datasheet" "~" (at 237.49 201.93 0)
+      (effects (font (size 1.27 1.27)) hide)
+    )
+    (pin "1")
+    (pin "2")
+    (instances
+      (project "weisse_cpu"
+        (path "/e63e39d7-6ac0-4ffd-8aa3-1841a4541b55"
+          (reference "R90") (unit 1)
+        )
+      )
+    )
+  )
   (symbol (lib_id "Device:LED") (at 345.44 344.17 0) (unit 1)
     (in_bom yes) (on_board yes) (dnp no) (fields_autoplaced)
@@
         (path "/e63e39d7-6ac0-4ffd-8aa3-1841a4541b55"
           (reference "LAUTSPRECHER1") (unit 1)
+        )
+      )
+    )
+  )
+  (symbol (lib_id "Device:R") (at 251.46 201.93 90) (unit 1)
+    (in_bom yes) (on_board yes) (dnp no) (fields_autoplaced)
+    (property "Reference" "R100" (at 251.46 195.58 90)
+      (effects (font (size 1.27 1.27)))
+    )
+    (property "Value" "R" (at 251.46 198.12 90)
+      (effects (font (size 1.27 1.27)))
+    )
+    (property "Footprint" "Resistor_THT:R_Axial_Power_L25.0mm_W9.0mm_P30.48mm" (at 251.46 203.708 90)
+      (effects (font (size 1.27 1.27)) hide)
+    )
+    (property "Datasheet" "~" (at 251.46 201.93 0)
+      (effects (font (size 1.27 1.27)) hide)
+    )
+    (pin "1")
+    (pin "2")
+    (instances
+      (project "weisse_cpu"
+        (path "/e63e39d7-6ac0-4ffd-8aa3-1841a4541b55"
+          (reference "R100") (unit 1)
         )
       )
@@
         )
       )
+    )
+  )
+  (symbol (lib_name "GND_2") (lib_id "power:GND") (at 355.6 31.75 90) (unit 1)
+    (in_bom yes) (on_board yes) (dnp no) (fields_autoplaced)
+    (property "Reference" "#PWR02" (at 361.95 31.75 0)
+      (effects (font (size 1.27 1.27)) hide)
+    )
+    (property "Value" "GND" (at 359.41 31.75 90)
+      (effects (font (size 1.27 1.27)) (justify right))
+    )
+    (property "Footprint" "" (at 355.6 31.75 0)
+      (effects (font (size 1.27 1.27)) hide)
+    )
+    (property "Datasheet" "" (at 355.6 31.75 0)
+      (effects (font (size 1.27 1.27)) hide)
+    )
+    (pin "1")
+    (instances
+      (project "weisse_cpu"
+        (path "/e63e39d7-6ac0-4ffd-8aa3-1841a4541b55"
+          (reference "#PWR02") (unit 1)
+        )
+      )

Commit message: zoom out
Parts:
- added R41, R65, R66: R, Resistor_THT:R_Axial_Power_L25.0mm_W6.4mm_P30.48mm, symbol Device:R
- R100, R90: footprint Resistor_THT:R_Axial_Power_L25.0mm_W9.0mm_P30.48mm -> Resistor_THT:R_Axial_Power_L25.0mm_W6.4mm_P30.48mm
Connections:
- new net: R41.2, R65.1, R66.1
Changed lines of the file:
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@@
   (junction (at 87.63 25.4) (diameter 0) (color 0 0 0 0)
   )
+  (junction (at 207.01 214.63) (diameter 0) (color 0 0 0 0)
+  )
   (junction (at 92.71 25.4) (diameter 0) (color 0 0 0 0)
   )
@@
     (stroke (width 0) (type default))
   )
+  (wire (pts (xy 207.01 201.93) (xy 207.01 214.63))
+    (stroke (width 0) (type default))
+  )
   (wire (pts (xy 176.53 45.72) (xy 182.88 45.72))
     (stroke (width 0) (type default))
@@
     (stroke (width 0) (type default))
   )
+  (wire (pts (xy 212.09 201.93) (xy 207.01 201.93))
+    (stroke (width 0) (type default))
+  )
   (wire (pts (xy 140.97 45.72) (xy 160.02 45.72))
     (stroke (width 0) (type default))
@@
   )
   (wire (pts (xy 102.87 45.72) (xy 121.92 45.72))
+    (stroke (width 0) (type default))
+  )
+  (wire (pts (xy 203.2 214.63) (xy 207.01 214.63))
+    (stroke (width 0) (type default))
+  )
+  (wire (pts (xy 207.01 214.63) (xy 212.09 214.63))
     (stroke (width 0) (type default))
   )
@@
         (path "/e63e39d7-6ac0-4ffd-8aa3-1841a4541b55"
           (reference "ICG10-1") (unit 2)
+        )
+      )
+    )
+  )
+  (symbol (lib_id "Device:R") (at 215.9 214.63 90) (unit 1)
+    (in_bom yes) (on_board yes) (dnp no) (fields_autoplaced)
+    (property "Reference" "R66" (at 215.9 208.28 90)
+      (effects (font (size 1.27 1.27)))
+    )
+    (property "Value" "R" (at 215.9 210.82 90)
+      (effects (font (size 1.27 1.27)))
+    )
+    (property "Footprint" "Resistor_THT:R_Axial_Power_L25.0mm_W6.4mm_P30.48mm" (at 215.9 216.408 90)
+      (effects (font (size 1.27 1.27)) hide)
+    )
+    (property "Datasheet" "~" (at 215.9 214.63 0)
+      (effects (font (size 1.27 1.27)) hide)
+    )
+    (pin "1")
+    (pin "2")
+    (instances
+      (project "weisse_cpu"
+        (path "/e63e39d7-6ac0-4ffd-8aa3-1841a4541b55"
+          (reference "R66") (unit 1)
         )
       )
@@
       (effects (font (size 1.27 1.27)))
     )
-    (property "Footprint" "Resistor_THT:R_Axial_Power_L25.0mm_W9.0mm_P30.48mm" (at 237.49 203.708 90)
+    (property "Footprint" "Resistor_THT:R_Axial_Power_L25.0mm_W6.4mm_P30.48mm" (at 237.49 203.708 90)
       (effects (font (size 1.27 1.27)) hide)
     )
@@
       (effects (font (size 1.27 1.27)))
     )
-    (property "Footprint" "Resistor_THT:R_Axial_Power_L25.0mm_W9.0mm_P30.48mm" (at 251.46 203.708 90)
+    (property "Footprint" "Resistor_THT:R_Axial_Power_L25.0mm_W6.4mm_P30.48mm" (at 251.46 203.708 90)
       (effects (font (size 1.27 1.27)) hide)
     )
@@
     )
   )
+  (symbol (lib_id "Device:R") (at 199.39 214.63 90) (unit 1)
+    (in_bom yes) (on_board yes) (dnp no) (fields_autoplaced)
+    (property "Reference" "R41" (at 199.39 208.28 90)
+      (effects (font (size 1.27 1.27)))
+    )
+    (property "Value" "R" (at 199.39 210.82 90)
+      (effects (font (size 1.27 1.27)))
+    )
+    (property "Footprint" "Resistor_THT:R_Axial_Power_L25.0mm_W6.4mm_P30.48mm" (at 199.39 216.408 90)
+      (effects (font (size 1.27 1.27)) hide)
+    )
+    (property "Datasheet" "~" (at 199.39 214.63 0)
+      (effects (font (size 1.27 1.27)) hide)
+    )
+    (pin "1")
+    (pin "2")
+    (instances
+      (project "weisse_cpu"
+        (path "/e63e39d7-6ac0-4ffd-8aa3-1841a4541b55"
+          (reference "R41") (unit 1)
+        )
+      )
+    )
+  )
   (symbol (lib_id "Connector:Conn_01x08_Male") (at 247.65 134.62 0) (unit 1)
     (in_bom yes) (on_board yes) (dnp no)
@@
         )
       )
+    )
+  )
+  (symbol (lib_id "Device:R") (at 215.9 201.93 90) (unit 1)
+    (in_bom yes) (on_board yes) (dnp no) (fields_autoplaced)
+    (property "Reference" "R65" (at 215.9 195.58 90)
+      (effects (font (size 1.27 1.27)))
+    )
+    (property "Value" "R" (at 215.9 198.12 90)
+      (effects (font (size 1.27 1.27)))
+    )
+    (property "Footprint" "Resistor_THT:R_Axial_Power_L25.0mm_W6.4mm_P30.48mm" (at 215.9 203.708 90)
+      (effects (font (size 1.27 1.27)) hide)
+    )
+    (property "Datasheet" "~" (at 215.9 201.93 0)
+      (effects (font (size 1.27 1.27)) hide)
+    )
+    (pin "1")
+    (pin "2")
+    (instances
+      (project "weisse_cpu"
+        (path "/e63e39d7-6ac0-4ffd-8aa3-1841a4541b55"
+          (reference "R65") (unit 1)
+        )
+      )

Commit message: fill got lost again
Parts:
- LED1, LED2, LED3, LED4, LED5: footprint LED_THT:LED_D3.0mm -> LED_THT:LED_D5.0mm
Connections:
- net GND: now also R100.1, R41.2, R65.1, R66.1, R90.2
Changed lines of the file:
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@@
   (junction (at 260.35 25.4) (diameter 0) (color 0 0 0 0)
   )
+  (junction (at 245.11 201.93) (diameter 0) (color 0 0 0 0)
+  )
   (junction (at 160.02 45.72) (diameter 0) (color 0 0 0 0)
   )
@@
     (stroke (width 0) (type default))
   )
-  (wire (pts (xy 241.3 201.93) (xy 247.65 201.93))
+  (wire (pts (xy 241.3 201.93) (xy 245.11 201.93))
+    (stroke (width 0) (type default))
+  )
+  (wire (pts (xy 245.11 201.93) (xy 247.65 201.93))
     (stroke (width 0) (type default))
   )
@@
       (effects (font (size 1.27 1.27)))
     )
-    (property "Footprint" "LED_THT:LED_D3.0mm" (at 345.44 313.69 0)
+    (property "Footprint" "LED_THT:LED_D5.0mm" (at 345.44 313.69 0)
       (effects (font (size 1.27 1.27)) hide)
     )
@@
       (effects (font (size 1.27 1.27)))
     )
-    (property "Footprint" "LED_THT:LED_D3.0mm" (at 345.44 354.33 0)
+    (property "Footprint" "LED_THT:LED_D5.0mm" (at 345.44 354.33 0)
       (effects (font (size 1.27 1.27)) hide)
     )
@@
       (effects (font (size 1.27 1.27)))
     )
-    (property "Footprint" "LED_THT:LED_D3.0mm" (at 345.44 344.17 0)
+    (property "Footprint" "LED_THT:LED_D5.0mm" (at 345.44 344.17 0)
       (effects (font (size 1.27 1.27)) hide)
     )
@@
       (effects (font (size 1.27 1.27)))
     )
-    (property "Footprint" "LED_THT:LED_D3.0mm" (at 345.44 335.28 0)
+    (property "Footprint" "LED_THT:LED_D5.0mm" (at 345.44 335.28 0)
       (effects (font (size 1.27 1.27)) hide)
     )
@@
       (effects (font (size 1.27 1.27)))
     )
-    (property "Footprint" "LED_THT:LED_D3.0mm" (at 345.44 323.85 0)
+    (property "Footprint" "LED_THT:LED_D5.0mm" (at 345.44 323.85 0)
       (effects (font (size 1.27 1.27)) hide)
     )
@@
     )
   )
+  (symbol (lib_name "GND_3") (lib_id "power:GND") (at 207.01 214.63 0) (unit 1)
+    (in_bom yes) (on_board yes) (dnp no) (fields_autoplaced)
+    (property "Reference" "#PWR03" (at 207.01 220.98 0)
+      (effects (font (size 1.27 1.27)) hide)
+    )
+    (property "Value" "GND" (at 207.01 219.71 0)
+      (effects (font (size 1.27 1.27)))
+    )
+    (property "Footprint" "" (at 207.01 214.63 0)
+      (effects (font (size 1.27 1.27)) hide)
+    )
+    (property "Datasheet" "" (at 207.01 214.63 0)
+      (effects (font (size 1.27 1.27)) hide)
+    )
+    (pin "1")
+    (instances
+      (project "weisse_cpu"
+        (path "/e63e39d7-6ac0-4ffd-8aa3-1841a4541b55"
+          (reference "#PWR03") (unit 1)
+        )
+      )
+    )
+  )
   (symbol (lib_id "Device:R_Pack08") (at 72.39 171.45 270) (unit 1)
     (in_bom yes) (on_board yes) (dnp no) (fields_autoplaced)
@@
         )
       )
+    )
+  )
+  (symbol (lib_name "GND_3") (lib_id "power:GND") (at 245.11 201.93 0) (unit 1)
+    (in_bom yes) (on_board yes) (dnp no) (fields_autoplaced)
+    (property "Reference" "#PWR04" (at 245.11 208.28 0)
+      (effects (font (size 1.27 1.27)) hide)
+    )
+    (property "Value" "GND" (at 245.11 207.01 0)
+      (effects (font (size 1.27 1.27)))
+    )
+    (property "Footprint" "" (at 245.11 201.93 0)
+      (effects (font (size 1.27 1.27)) hide)
+    )
+    (property "Datasheet" "" (at 245.11 201.93 0)
+      (effects (font (size 1.27 1.27)) hide)
+    )
+    (pin "1")
+    (instances
+      (project "weisse_cpu"
+        (path "/e63e39d7-6ac0-4ffd-8aa3-1841a4541b55"
+          (reference "#PWR04") (unit 1)
+        )
+      )

Commit message: schaltplan
Connections:
- net +12V: now also EINGAENGE1.1 (Pin_1), LAUTSPRECHER1.2 (Pin_2), LEUCHTZIFFERNANZEIGE1.4 (Pin_4), MUENZANNAHME1.4 (Pin_4), SERIELLE_DATEN1.8 (Pin_8), TASTEN1.6 (Pin_6), TUERSCHALTER+SPIELZAEHLER1.3 (Pin_3), ZUSATZTASTEN1.2 (Pin_2)
- net +24V: now also LAUTSPRECHER1.1 (Pin_1), MUENZANNAHME1.2 (Pin_2), SERIELLE_DATEN1.4 (Pin_4), WALZENANSTEUERUNG1.12 (Pin_12)
- net +48V: now also AUSWERFER+SPERRMAG1.1 (Pin_1), EINGAENGE1.6 (Pin_6), SERIELLE_DATEN1.2 (Pin_2), TUERSCHALTER+SPIELZAEHLER1.4 (Pin_4), WALZENANSTEUERUNG1.14 (Pin_14)
- net +5V: now also LEUCHTZIFFERNANZEIGE1.3 (Pin_3), SERIELLE_DATEN1.1 (Pin_1)
- net GND: now also ICC6.16 (GND), ICD6.14 (GND), ICE6.14 (GND), ICK11.11 (V-), LEUCHTZIFFERNANZEIGE1.1 (Pin_1), ZUSATZTASTEN1.1 (Pin_1); no longer LEISTUNGSAUSGAENGE1.2 (Pin_2), LEISTUNGSNETZ1.1 (Pin_1), LEISTUNGSNETZ1.2 (Pin_2), LEISTUNGSNETZ1.3 (Pin_3), R100.1, R41.2, R65.1, R66.1, R90.2
- net GNDPWR: now reaches SERIELLE_DATEN1.7 (Pin_7)
- net GNDPWR: now also LAUTSPRECHER1.4 (Pin_4), LEISTUNGSAUSGAENGE1.2 (Pin_2), LEISTUNGSNETZ1.1 (Pin_1), LEISTUNGSNETZ1.2 (Pin_2), LEISTUNGSNETZ1.3 (Pin_3), MUENZANNAHME1.1 (Pin_1), R100.1, R41.2, R65.1, R66.1, R90.2, WALZENANSTEUERUNG1.13 (Pin_13)
- net at LAMPENZEILEN1.1 (Pin_1): now also LAMPENZEILEN1.2 (Pin_2)
- net at LAMPENZEILEN1.10 (Pin_10): now also LAMPENZEILEN1.9 (Pin_9)
- net at LAMPENZEILEN1.11 (Pin_11): now also LAMPENZEILEN1.12 (Pin_12)
- net at LAMPENZEILEN1.13 (Pin_13): now also LAMPENZEILEN1.14 (Pin_14)
- net at LAMPENZEILEN1.15 (Pin_15): now also LAMPENZEILEN1.16 (Pin_16)
- net at LAMPENZEILEN1.3 (Pin_3): now also LAMPENZEILEN1.4 (Pin_4)
- net at LAMPENZEILEN1.5 (Pin_5): now also LAMPENZEILEN1.6 (Pin_6)
- net at LAMPENZEILEN1.7 (Pin_7): now also LAMPENZEILEN1.8 (Pin_8)
Other:
- moved on the sheet: LEUCHTZIFFERNANZEIGE1

Commit message: walz
Parts:
- added ICG1, ICH2: LM324, Package_DIP:DIP-14_W7.62mm, symbol Amplifier_Operational:LM324
- added ICH1: 4098, Package_DIP:DIP-16_W7.62mm, symbol 4xxx:4098
Other:
- moved on the sheet: ICC6, ICD6, ICE6, SW1, WALZENANSTEUERUNG1

Commit message: thyristor
Parts:
- added D1, D10, D11, D12, D13, D2, D25, D26: D, Diode_THT:D_A-405_P7.62mm_Horizontal, symbol Device:D
- added D27, D3: D, Diode_THT:D_DO-27_P15.24mm_Horizontal, symbol Device:D
- added TY1, TY15, TY16, TY2, TY5, TY6, TY7, TY8: TIC126, Package_TO_SOT_THT:TO-220-3_Vertical, symbol Triac_Thyristor:TIC126
Connections:
- net at R40.1, TR1.3 (E), TR10.3 (E)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: now also D1.1 (K), D10.1 (K), D11.1 (K), D12.1 (K), D13.1 (K), D2.1 (K), D25.1 (K), D26.1 (K)
- new net: D1.2 (A), D10.2 (A), D11.2 (A), D12.2 (A), D13.2 (A), D2.2 (A), D25.2 (A), D26.2 (A)
Other:
- moved on the sheet: ICG10-1B, ICG10-1C, ICG10-1D, ICG10-1E, ICK11A, ICK11B, ICK11C, ICK11D, ICK11E, LAMPENZEILEN1, RM81, SERVICEANZEIGE+TASTATUR1
