File: weisse_cpu.kicad_sch (KiCad schematic)
At the start: 77 parts, among them SW1 SW_DIP_x04

Commit message: thryrrristorrr
Parts:
- ICC6: value 628128_DIP32_SSOP32 -> CXK5816PN-12L; symbol Memory_RAM:628128_DIP32_SSOP32 -> Memory_RAM:CXK5816PN
Connections:
- net GND: now also ICC6.12 (GND); no longer ICC6.16 (GND)
Changed lines of the file:
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@@
     )
   )
-  (symbol (lib_name "GND_4") (lib_id "power:GND") (at 184.15 391.16 0) (unit 1)
-    (in_bom yes) (on_board yes) (dnp no) (fields_autoplaced)
-    (property "Reference" "#PWR019" (at 184.15 397.51 0)
-      (effects (font (size 1.27 1.27)) hide)
-    )
-    (property "Value" "GND" (at 184.15 396.24 0)
-      (effects (font (size 1.27 1.27)))
-    )
-    (property "Footprint" "" (at 184.15 391.16 0)
-      (effects (font (size 1.27 1.27)) hide)
-    )
-    (property "Datasheet" "" (at 184.15 391.16 0)
+  (symbol (lib_name "GND_4") (lib_id "power:GND") (at 181.61 377.19 0) (unit 1)
+    (in_bom yes) (on_board yes) (dnp no) (fields_autoplaced)
+    (property "Reference" "#PWR019" (at 181.61 383.54 0)
+      (effects (font (size 1.27 1.27)) hide)
+    )
+    (property "Value" "GND" (at 181.61 382.27 0)
+      (effects (font (size 1.27 1.27)))
+    )
+    (property "Footprint" "" (at 181.61 377.19 0)
+      (effects (font (size 1.27 1.27)) hide)
+    )
+    (property "Datasheet" "" (at 181.61 377.19 0)
       (effects (font (size 1.27 1.27)) hide)
     )
@@
     )
   )
-  (symbol (lib_id "Memory_RAM:628128_DIP32_SSOP32") (at 184.15 365.76 0) (unit 1)
-    (in_bom yes) (on_board yes) (dnp no) (fields_autoplaced)
-    (property "Reference" "ICC6" (at 186.3441 337.82 0)
-      (effects (font (size 1.27 1.27)) (justify left))
-    )
-    (property "Value" "628128_DIP32_SSOP32" (at 186.3441 340.36 0)
-      (effects (font (size 1.27 1.27)) (justify left))
-    )
-    (property "Footprint" "Package_DIP:DIP-24_W15.24mm" (at 184.15 365.76 0)
-      (effects (font (size 1.27 1.27)) hide)
-    )
-    (property "Datasheet" "http://www.futurlec.com/Datasheet/Memory/628128.pdf" (at 184.15 365.76 0)
+  (symbol (lib_id "Memory_RAM:CXK5816PN") (at 181.61 364.49 0) (unit 1)
+    (in_bom yes) (on_board yes) (dnp no) (fields_autoplaced)
+    (property "Reference" "ICC6" (at 183.8041 336.55 0)
+      (effects (font (size 1.27 1.27)) (justify left))
+    )
+    (property "Value" "CXK5816PN-12L" (at 183.8041 339.09 0)
+      (effects (font (size 1.27 1.27)) (justify left))
+    )
+    (property "Footprint" "Package_DIP:DIP-24_W15.24mm" (at 181.61 364.49 0)
+      (effects (font (size 1.27 1.27)) hide)
+    )
+    (property "Datasheet" "https://pdf1.alldatasheet.com/datasheet-pdf/view/154355/SONY/CXK5816PN.html" (at 181.61 364.49 0)
       (effects (font (size 1.27 1.27)) hide)
     )
     (pin "16")
-    (pin "32")
     (pin "1")
     (pin "10")
@@
     (pin "23")
     (pin "24")
-    (pin "25")
-    (pin "26")
-    (pin "27")
-    (pin "28")
-    (pin "29")
-    (pin "3")
-    (pin "30")
-    (pin "31")
-    (pin "4")
-    (pin "5")
+    (pin "3")
+    (pin "4")
+    (pin "5")

Commit message: ram
Parts:
- TR32: footprint Package_TO_SOT_THT:TO-220-3_Vertical -> Package_TO_SOT_THT:TO-126-3_Vertical
Changed lines of the file:
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@@
       (effects (font (size 1.27 1.27)) (justify left))
     )
-    (property "Footprint" "Package_TO_SOT_THT:TO-220-3_Vertical" (at 69.85 73.66 0)
+    (property "Footprint" "Package_TO_SOT_THT:TO-126-3_Vertical" (at 69.85 73.66 0)
       (effects (font (size 1.27 1.27)) hide)
     )

Commit message: batterie
Parts:
- added RN1: R_Pack08, Package_DIP:DIP-16_W7.62mm, symbol Device:R_Pack08
- BATTERIE2: footprint Battery:BatteryHolder_Keystone_2460_1xAA -> Library:Batterie
Connections:
- net +48V: now also GONG1.1 (Pin_1)
- net at TASTEN1.1 (Pin_1): now also RN1.2 (R2.1)
- net at TASTEN1.2 (Pin_2): now also RN1.3 (R3.1)
- net at TASTEN1.3 (Pin_3): now also RN1.4 (R4.1)
- net at TASTEN1.4 (Pin_4): now also RN1.5 (R5.1)
- net A0: now reaches ICE6.10 (A0)
- net A0: now also ICC6.8 (A0), ICD6.10 (A0)
- net D0: now reaches ICE6.11 (D0)
- net D0: now also ICC6.9 (I/O1), ICD6.11 (D0)
- net D1: now reaches ICE6.12 (D1)
- net D1: now also ICC6.10 (I/O2), ICD6.12 (D1)
- net D2: now reaches ICE6.13 (D2)
- net D2: now also ICC6.11 (I/O3), ICD6.13 (D2)
- net D3: now reaches ICE6.15 (D3)
- net D3: now also ICC6.13 (I/O4), ICD6.15 (D3)
- net D4: now reaches ICE6.16 (D4)
- net D4: now also ICC6.14 (I/O5), ICD6.16 (D4)
- net D5: now reaches ICE6.17 (D5)
- net D5: now also ICC6.15 (I/O6), ICD6.17 (D5)
- net D6: now reaches ICE6.18 (D6)
- net D6: now also ICC6.16 (I/O7), ICD6.18 (D6)
- net D7: now reaches ICE6.19 (D7)
- net D7: now also ICC6.17 (I/O8), ICD6.19 (D7)
- net A12: now reaches ICE6.2 (A12)
- net A12: now also ICD6.2 (A12)
- net A10: now reaches ICE6.21 (A10)
- net A10: now also ICC6.19 (A10), ICD6.21 (A10)
- net A11: now reaches ICE6.23 (A11)
- net A11: now also ICD6.23 (A11)
- net A9: now reaches ICE6.24 (A9)
- net A9: now also ICC6.22 (A9), ICD6.24 (A9)
- net A8: now reaches ICE6.25 (A8)
- net A8: now also ICC6.23 (A8), ICD6.25 (A8)
- net A13: now reaches ICE6.26 (A13)
- net A13: now also ICD6.26 (A13)
- net A7: now reaches ICE6.3 (A7)
- net A7: now also ICC6.1 (A7), ICD6.3 (A7)
- net A6: now reaches ICE6.4 (A6)
- net A6: now also ICC6.2 (A6), ICD6.4 (A6)
- net A5: now reaches ICE6.5 (A5)
- net A5: now also ICC6.3 (A5), ICD6.5 (A5)
- net A4: now reaches ICE6.6 (A4)
- net A4: now also ICC6.4 (A4), ICD6.6 (A4)
- net A3: now reaches ICE6.7 (A3)
- net A3: now also ICC6.5 (A3), ICD6.7 (A3)
- net A2: now reaches ICE6.8 (A2)
- net A2: now also ICC6.6 (A2), ICD6.8 (A2)
- net A1: now reaches ICE6.9 (A1)
- net A1: now also ICC6.7 (A1), ICD6.9 (A1)
Other:
- moved on the sheet: TASTEN1

Commit message: muenzen
Parts:
- added RM10, RM4, RM8, RM83, RM85: R_Pack08, Package_DIP:DIP-16_W7.62mm, symbol Device:R_Pack08
- renumbered RN1 to RM6
Connections:
- net at MUENZANNAHME1.10 (Pin_10): now also RM83.4 (R4.1)
- net at MUENZANNAHME1.11 (Pin_11): now also RM83.3 (R3.1)
- net at MUENZANNAHME1.12 (Pin_12): now also RM83.2 (R2.1)
- net at MUENZANNAHME1.13 (Pin_13): now also RM83.1 (R1.1)
- net at MUENZANNAHME1.14 (Pin_14): now also RM85.4 (R4.1)
- net at MUENZANNAHME1.15 (Pin_15): now also RM85.5 (R5.1)
- net at MUENZANNAHME1.16 (Pin_16): now also RM85.6 (R6.1)
- net at MUENZANNAHME1.17 (Pin_17): now also RM85.7 (R7.1)
- net at MUENZANNAHME1.18 (Pin_18): now also RM85.8 (R8.1)
- net at MUENZANNAHME1.6 (Pin_6): now also RM83.8 (R8.1)
- net at MUENZANNAHME1.7 (Pin_7): now also RM83.7 (R7.1)
- net at MUENZANNAHME1.8 (Pin_8): now also RM83.6 (R6.1)
- net at MUENZANNAHME1.9 (Pin_9): now also RM83.5 (R5.1)
- net at WALZENANSTEUERUNG1.2 (Pin_2): now also RM4.14 (R3.2)
- net at WALZENANSTEUERUNG1.3 (Pin_3): now also RM4.13 (R4.2)
- net at WALZENANSTEUERUNG1.4 (Pin_4): now also RM4.12 (R5.2)
- net at ZUSATZTASTEN1.5 (Pin_5): now also RM8.10 (R7.2)
- net at ZUSATZTASTEN1.6 (Pin_6): now also RM8.14 (R3.2)
Other:
- moved on the sheet: MUENZANNAHME1, SERIELLE_DATEN1, ZUSATZTASTEN1

Commit message: logic
Parts:
- added ICB4: 74LS245, Package_DIP:DIP-20_W7.62mm, symbol 74xx:74LS245
- added ICC3: 74LS04, Package_DIP:DIP-14_W7.62mm, symbol 74xx:74LS04
- added ICD3: 74LS257, Package_DIP:DIP-16_W7.62mm, symbol 74xx:74LS257
- added Q1: Crystal, Crystal:Crystal_AT310_D3.0mm_L10.0mm_Vertical, symbol Device:Crystal
- added Q2: Crystal, Crystal:Crystal_HC18-U_Vertical, symbol Device:Crystal

Commit message: cpu
Parts:
- added ICB2: 8085, Package_DIP:DIP-40_W15.24mm, symbol 8085:8085
Connections:
- net GND: now also ICB2.20 (GND)
- new net VCC: ICB2.40 (VCC)
Other:
- moved on the sheet: SW1
Changed lines of the file:
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@@
+    )
+  )
+  (symbol (lib_id "8085:8085") (at 226.06 356.87 0) (unit 1)
+    (in_bom yes) (on_board yes) (dnp no) (fields_autoplaced)
+    (property "Reference" "ICB2" (at 226.06 308.61 0)
+      (effects (font (size 1.524 1.524)))
+    )
+    (property "Value" "8085" (at 226.06 311.15 0)
+      (effects (font (size 1.524 1.524)))
+    )
+    (property "Footprint" "Package_DIP:DIP-40_W15.24mm" (at 226.06 355.6 0)
+      (effects (font (size 1.524 1.524)) hide)
+    )
+    (property "Datasheet" "" (at 226.06 355.6 0)
+      (effects (font (size 1.524 1.524)))
+    )
+    (pin "1")
+    (pin "10")
+    (pin "11")
+    (pin "12")
+    (pin "13")
+    (pin "14")
+    (pin "15")
+    (pin "16")
+    (pin "17")
+    (pin "18")
+    (pin "19")
+    (pin "2")
+    (pin "20")
+    (pin "21")
+    (pin "22")
+    (pin "23")
+    (pin "24")
+    (pin "25")
+    (pin "26")
+    (pin "27")
+    (pin "28")
+    (pin "29")
+    (pin "3")
+    (pin "30")
+    (pin "31")
+    (pin "32")
+    (pin "33")
+    (pin "34")
+    (pin "35")
+    (pin "36")
+    (pin "37")
+    (pin "38")
+    (pin "39")
+    (pin "4")
+    (pin "40")
+    (pin "5")
+    (pin "6")
+    (pin "7")
+    (pin "8")
+    (pin "9")
+    (instances
+      (project "weisse_cpu"
+        (path "/e63e39d7-6ac0-4ffd-8aa3-1841a4541b55"
+          (reference "ICB2") (unit 1)
+        )
+      )
     )
   )
@@
     )
   )
-  (symbol (lib_id "Switch:SW_DIP_x04") (at 255.27 379.73 0) (unit 1)
+  (symbol (lib_id "Switch:SW_DIP_x04") (at 267.97 350.52 0) (unit 1)
     (in_bom yes) (on_board yes) (dnp no) (fields_autoplaced)
-    (property "Reference" "SW1" (at 255.27 367.03 0)
+    (property "Reference" "SW1" (at 267.97 337.82 0)
       (effects (font (size 1.27 1.27)))
     )
-    (property "Value" "SW_DIP_x04" (at 255.27 369.57 0)
+    (property "Value" "SW_DIP_x04" (at 267.97 340.36 0)
       (effects (font (size 1.27 1.27)))
     )
-    (property "Footprint" "Button_Switch_THT:SW_DIP_SPSTx04_Slide_9.78x12.34mm_W7.62mm_P2.54mm" (at 255.27 379.73 0)
+    (property "Footprint" "Button_Switch_THT:SW_DIP_SPSTx04_Slide_9.78x12.34mm_W7.62mm_P2.54mm" (at 267.97 350.52 0)
       (effects (font (size 1.27 1.27)) hide)
     )
-    (property "Datasheet" "~" (at 255.27 379.73 0)
+    (property "Datasheet" "~" (at 267.97 350.52 0)
       (effects (font (size 1.27 1.27)) hide)
     )

Commit message: rtx 4060
Parts:
- added C159, C160, C161: C, Capacitor_THT:C_Rect_L9.0mm_W2.5mm_P7.50mm_MKT, symbol Device:C
- added ICB10, ICB9, ICC10, ICD10, ICE10, ICF10: 4066, Package_DIP:DIP-14_W7.62mm, symbol 4xxx:4066

Commit message: transistoren
Parts:
- added ICB5: 74LS373, Package_DIP:DIP-20_W7.62mm, symbol 74xx:74LS373
- added ICD8, ICF8: CD4051B, Package_DIP:DIP-16_W7.62mm, symbol Analog_Switch:CD4051B
- added TR70, TR71, TR72, TR73, TR80, TR81, TR82, TR83, TR95, TR96, TR97: Q_NPN_Darlington_BCE, Package_TO_SOT_THT:TO-220-3_Vertical, symbol Device:Q_NPN_Darlington_BCE
Connections:
- net GND: now also ICB4.10 (GND), ICC3.7 (GND), ICD3.8 (GND), ICH1.8 (VSS), ICB5.10 (GND)
- new net: TR70.3 (E), TR71.3 (E), TR72.3 (E), TR73.3 (E), TR80.3 (E), TR81.3 (E)
- new net: TR82.3 (E), TR83.3 (E), TR95.3 (E), TR96.3 (E)
Other:
- moved on the sheet: ICD3
