File: weisse_cpu.kicad_sch (KiCad schematic)
At the start: 112 parts, among them Q1 Crystal, Q2 Crystal, SW1 SW_DIP_x04

Commit message: caps
Parts:
- added C20, C21, C22, C23, C24, C25, C26, C27: C, Capacitor_THT:C_Rect_L7.0mm_W2.0mm_P5.00mm, symbol Device:C
- added ICA7: 4066, Package_DIP:DIP-14_W7.62mm, symbol 4xxx:4066
- added ICE2: 8256, Package_DIP:DIP-40_W15.24mm, symbol 8085:8256
- added ICF3: 4028, Package_DIP:DIP-16_W7.62mm, symbol 4xxx:4028
- added R29: R, Resistor_THT:R_Axial_DIN0414_L11.9mm_D4.5mm_P20.32mm_Horizontal, symbol Device:R
- renumbered R29 to R28
Other:
- moved on the sheet: BATTERIE2, SW1

Commit message: chips
Parts:
- added ICG10-2, ICH10: 4066, Package_DIP:DIP-14_W7.62mm, symbol 4xxx:4066
- added ICG8-1: 74LS290, Package_DIP:DIP-14_W7.62mm, symbol 74xx:74LS290
- added ICG8-2: 4040, Package_DIP:DIP-16_W7.62mm, symbol 4xxx:4040
- added ICL10: NE556, Package_DIP:DIP-14_W7.62mm, symbol Timer:NE556
- added ICL8: 4013, Package_DIP:DIP-14_W7.62mm, symbol 4xxx:4013
- added ICL9: 4093, Package_DIP:DIP-14_W7.62mm, symbol 4xxx_IEEE:4093

Commit message: traces
Connections:
- net +24V: now also LEISTUNGSAUSGAENGE1.10 (Pin_10)
Changed lines of the file:
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@@
+    (stroke (width 0) (type default))
+  )
+  (wire (pts (xy 346.71 52.07) (xy 355.6 52.07))
     (stroke (width 0) (type default))
   )
@@
         )
       )
+    )
+  )
+  (symbol (lib_id "power:+24V") (at 355.6 52.07 270) (unit 1)
+    (in_bom yes) (on_board yes) (dnp no) (fields_autoplaced)
+    (property "Reference" "#PWR041" (at 351.79 52.07 0)
+      (effects (font (size 1.27 1.27)) hide)
+    )
+    (property "Value" "+24V" (at 359.41 52.07 90)
+      (effects (font (size 1.27 1.27)) (justify left))
+    )
+    (property "Footprint" "" (at 355.6 52.07 0)
+      (effects (font (size 1.27 1.27)) hide)
+    )
+    (property "Datasheet" "" (at 355.6 52.07 0)
+      (effects (font (size 1.27 1.27)) hide)
+    )
+    (pin "1")
+    (instances
+      (project "weisse_cpu"
+        (path "/e63e39d7-6ac0-4ffd-8aa3-1841a4541b55"
+          (reference "#PWR041") (unit 1)
+        )
+      )

Commit message: lm324
Parts:
- added ICC4: 74LS00, Package_DIP:DIP-14_W7.62mm, symbol 74xx:74LS00
- added ICD4: 74LS244, Package_DIP:DIP-20_W7.62mm, symbol 74xx:74LS244
- added ICE5, ICF5: 74LS42, Package_DIP:DIP-16_W7.62mm, symbol 74xx:74LS42
- added ICF2, ICG2, ICG4, ICG4-1, ICK6: LM324, Package_DIP:DIP-14_W7.62mm, symbol Amplifier_Operational:LM324
- added ICG5: ~, Package_DIP:DIP-40_W15.24mm, symbol 8085:8279
- added ICH5: 74LS138, Package_DIP:DIP-16_W7.62mm, symbol 74xx:74LS138
- added ICH6: 74HC237, Package_DIP:DIP-20_W7.62mm, symbol 74xx:74HC273
- added R4: R, Resistor_THT:R_Axial_DIN0204_L3.6mm_D1.6mm_P7.62mm_Horizontal, symbol Device:R
- added RM50, RM56, RM57, RM66: R_Network08, Resistor_THT:R_Array_SIP9, symbol Device:R_Network08
Connections:
- net GND: now also ICB10.7 (VSS), ICB9.7 (VSS), ICC10.7 (VSS), ICD10.7 (VSS), ICE10.7 (VSS), ICF10.7 (VSS), ICG10-1.14 (VDD), ICG10-2.7 (VSS), ICG8-1.7 (GND), ICG8-2.8 (VSS), ICH10.7 (VSS), ICL10.7 (GND), ICL10.7 (GND), ICL8.7 (VSS), ICL9.7 (Vss), ICL9.7 (Vss), ICG5.20 (Vss)
- net at ICG1.14: now also WALZENANSTEUERUNG1.15 (Pin_15)
- new net: ICF2.14, R4.1
Other:
- moved on the sheet: ICB4, ICG1A, ICG1B, ICG1C, ICG1D, ICG1E, ICH1A, ICH1B, ICH2A, ICH2B, ICH2C, ICH2D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

Commit message: erthjerghse
Parts:
- removed ICH6: 74HC237, Package_DIP:DIP-20_W7.62mm, symbol 74xx:74HC273
- added C1, C76: C, Capacitor_THT:C_Rect_L9.0mm_W2.5mm_P7.50mm_MKT, symbol Device:C
- added ICH6, ICJ5, ICJ6: 74AHC273, Package_DIP:DIP-20_W7.62mm, symbol 74xx:74AHC273
- added ICK5: LM324, Package_DIP:DIP-14_W7.62mm, symbol Amplifier_Operational:LM324
- added R3: R, Resistor_THT:R_Axial_DIN0204_L3.6mm_D1.6mm_P7.62mm_Horizontal, symbol Device:R
- added RM20, RM5: R_Network04, Resistor_THT:R_Array_SIP5, symbol Device:R_Network04
- added RN1: R_Network08, Resistor_THT:R_Array_SIP9, symbol Device:R_Network08
Connections:
- net GND: now also BATTERIE2.2 (-)
- net at TY8.1 (K): now also TY15.1 (K), TY16.1 (K), TY7.1 (K)
- net at TY1.1 (K): now also TY2.1 (K), TY5.1 (K), TY6.1 (K)

Commit message: caps
Parts:
- added C10, C11, C4, C5, C6, C7, C8, C9: C, Capacitor_THT:C_Axial_L3.8mm_D2.6mm_P7.50mm_Horizontal, symbol Device:C
- added C2, C3: C, Capacitor_THT:CP_Radial_Tantal_D4.5mm_P2.50mm, symbol Device:C
- added RM3: R_Network08, Resistor_THT:R_Array_SIP9, symbol Device:R_Network08
- renumbered RM5 to RM2
Connections:
- new net: C6.1, RM3.3 (R2)
- new net: C5.1, RM3.2 (R1)
- new net: C7.1, RM3.4 (R3)
- new net: C8.1, RM3.5 (R4)
- new net: C11.1, RM3.8 (R7)

Commit message: 12v cap
Parts:
- added D14, D15, D16, D17, D28, D29, D4, D5: D, Diode_THT:D_A-405_P7.62mm_Horizontal, symbol Device:D
Connections:
- net +12V: now also C161.1
- net GND: now also C161.2
- net at TY8.2 (A): now also LAMPENZEILEN1.11 (Pin_11), LAMPENZEILEN1.12 (Pin_12), D17.2 (A)
- net at TY16.2 (A): now also LAMPENZEILEN1.15 (Pin_15), LAMPENZEILEN1.16 (Pin_16), D29.2 (A)
- net at TY15.2 (A): now also LAMPENZEILEN1.13 (Pin_13), LAMPENZEILEN1.14 (Pin_14), D28.2 (A)
- net at LAMPENZEILEN1.1 (Pin_1), LAMPENZEILEN1.2 (Pin_2): now also TY1.2 (A), D4.2 (A)
- net at LAMPENZEILEN1.10 (Pin_10), LAMPENZEILEN1.9 (Pin_9): now also TY7.2 (A), D16.2 (A)
- net at LAMPENZEILEN1.3 (Pin_3), LAMPENZEILEN1.4 (Pin_4): now also TY2.2 (A), D5.2 (A)
- net at LAMPENZEILEN1.5 (Pin_5), LAMPENZEILEN1.6 (Pin_6): now also TY5.2 (A), D14.2 (A)
- net at LAMPENZEILEN1.7 (Pin_7), LAMPENZEILEN1.8 (Pin_8): now also TY6.2 (A), D15.2 (A)
- new net: D14.1 (K), D15.1 (K), D16.1 (K), D17.1 (K), D28.1 (K), D29.1 (K), D4.1 (K), D5.1 (K)
Other:
- moved on the sheet: LAMPENZEILEN1

Commit message: power resistors
Parts:
- D27, D3: footprint Diode_THT:D_DO-27_P15.24mm_Horizontal -> BigOnes:BigDiode
- R100, R41, R65, R66, R90: footprint Resistor_THT:R_Axial_Power_L25.0mm_W6.4mm_P30.48mm -> BigOnes:BigResistor
- R40: footprint Resistor_THT:R_Axial_Power_L20.0mm_W6.4mm_P30.48mm -> BigOnes:BigResistor
Connections:
- net at D27.1 (K): now also D3.1 (K)
Changed lines of the file:
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@@
     (stroke (width 0) (type default))
   )
+  (wire (pts (xy 73.66 95.25) (xy 73.66 90.17))
+    (stroke (width 0) (type default))
+  )
   (wire (pts (xy 123.19 111.76) (xy 125.73 111.76))
     (stroke (width 0) (type default))
@@
     (stroke (width 0) (type default))
   )
+  (wire (pts (xy 73.66 90.17) (xy 88.9 90.17))
+    (stroke (width 0) (type default))
+  )
   (wire (pts (xy 560.07 210.82) (xy 548.64 210.82))
     (stroke (width 0) (type default))
@@
     (stroke (width 0) (type default))
   )
+  (wire (pts (xy 88.9 90.17) (xy 88.9 95.25))
+    (stroke (width 0) (type default))
+  )
   (wire (pts (xy 560.07 218.44) (xy 523.24 218.44))
     (stroke (width 0) (type default))
@@
       (effects (font (size 1.27 1.27)))
     )
-    (property "Footprint" "Resistor_THT:R_Axial_Power_L25.0mm_W6.4mm_P30.48mm" (at 215.9 216.408 90)
+    (property "Footprint" "BigOnes:BigResistor" (at 215.9 216.408 90)
       (effects (font (size 1.27 1.27)) hide)
     )
@@
       (effects (font (size 1.27 1.27)))
     )
-    (property "Footprint" "Resistor_THT:R_Axial_Power_L20.0mm_W6.4mm_P30.48mm" (at 172.72 47.498 90)
+    (property "Footprint" "BigOnes:BigResistor" (at 172.72 47.498 90)
       (effects (font (size 1.27 1.27)) hide)
     )
@@
       (effects (font (size 1.27 1.27)))
     )
-    (property "Footprint" "Diode_THT:D_DO-27_P15.24mm_Horizontal" (at 92.71 95.25 0)
+    (property "Footprint" "BigOnes:BigDiode" (at 92.71 95.25 0)
       (effects (font (size 1.27 1.27)) hide)
     )
@@
       (effects (font (size 1.27 1.27)))
     )
-    (property "Footprint" "Resistor_THT:R_Axial_Power_L25.0mm_W6.4mm_P30.48mm" (at 237.49 203.708 90)
+    (property "Footprint" "BigOnes:BigResistor" (at 237.49 203.708 90)
       (effects (font (size 1.27 1.27)) hide)
     )
@@
       (effects (font (size 1.27 1.27)))
     )
-    (property "Footprint" "Resistor_THT:R_Axial_Power_L25.0mm_W6.4mm_P30.48mm" (at 251.46 203.708 90)
+    (property "Footprint" "BigOnes:BigResistor" (at 251.46 203.708 90)
       (effects (font (size 1.27 1.27)) hide)
     )
@@
       (effects (font (size 1.27 1.27)))
     )
-    (property "Footprint" "Resistor_THT:R_Axial_Power_L25.0mm_W6.4mm_P30.48mm" (at 199.39 216.408 90)
+    (property "Footprint" "BigOnes:BigResistor" (at 199.39 216.408 90)
       (effects (font (size 1.27 1.27)) hide)
     )
@@
       (effects (font (size 1.27 1.27)))
     )
-    (property "Footprint" "Resistor_THT:R_Axial_Power_L25.0mm_W6.4mm_P30.48mm" (at 215.9 203.708 90)
+    (property "Footprint" "BigOnes:BigResistor" (at 215.9 203.708 90)
       (effects (font (size 1.27 1.27)) hide)
     )
@@
       (effects (font (size 1.27 1.27)))
     )
-    (property "Footprint" "Diode_THT:D_DO-27_P15.24mm_Horizontal" (at 77.47 95.25 0)
+    (property "Footprint" "BigOnes:BigDiode" (at 77.47 95.25 0)
       (effects (font (size 1.27 1.27)) hide)
     )
