File: tester/tester.kicad_pcb (KiCad board)
At the start: 2 copper layers, 36.8 x 92.7 mm, 70 parts

Commit message: reorg
Parts:
- moved RN2 9.66 mm to (227.5, 85.2)
- moved RN1 8.07 mm to (227.5, 63.6)
- moved RN4 7.34 mm to (227.8, 128.3)
- moved RN3 6.22 mm to (227.5, 92.8)
Connections:
- D11 pad 1: Net-(D11-K) -> Net-(D10-K)
- D11 pad 2: Net-(D10-A) -> Net-(D11-A)
- D12 pad 1: Net-(D12-K) -> Net-(D10-K)
- D12 pad 2: Net-(D10-A) -> Net-(D12-A)
- D13 pad 1: Net-(D13-K) -> Net-(D10-K)
- D13 pad 2: Net-(D10-A) -> Net-(D13-A)
- D14 pad 1: Net-(D14-K) -> Net-(D10-K)
- D14 pad 2: Net-(D10-A) -> Net-(D14-A)
- D15 pad 1: Net-(D15-K) -> Net-(D10-K)
- D15 pad 2: Net-(D10-A) -> Net-(D15-A)
- D16 pad 1: Net-(D16-K) -> Net-(D10-K)
- D16 pad 2: Net-(D10-A) -> Net-(D16-A)
- D17 pad 1: Net-(D1-K) -> Net-(D17-K)
- D17 pad 2: Net-(D17-A) -> Net-(D1-A)
- D18 pad 1: Net-(D10-K) -> Net-(D17-K)
- D18 pad 2: Net-(D17-A) -> Net-(D10-A)
- D19 pad 1: Net-(D11-K) -> Net-(D17-K)
- D19 pad 2: Net-(D17-A) -> Net-(D11-A)
- D2 pad 1: Net-(D10-K) -> Net-(D1-K)
- D2 pad 2: Net-(D1-A) -> Net-(D10-A)
- D20 pad 1: Net-(D12-K) -> Net-(D17-K)
- D20 pad 2: Net-(D17-A) -> Net-(D12-A)
- D21 pad 1: Net-(D13-K) -> Net-(D17-K)
- D21 pad 2: Net-(D17-A) -> Net-(D13-A)
- D22 pad 1: Net-(D14-K) -> Net-(D17-K)
- D22 pad 2: Net-(D17-A) -> Net-(D14-A)
- D23 pad 1: Net-(D15-K) -> Net-(D17-K)
- D23 pad 2: Net-(D17-A) -> Net-(D15-A)
- D24 pad 1: Net-(D16-K) -> Net-(D17-K)
- D24 pad 2: Net-(D17-A) -> Net-(D16-A)
- D25 pad 1: Net-(D1-K) -> Net-(D25-K)
- D25 pad 2: Net-(D25-A) -> Net-(D1-A)
- D26 pad 1: Net-(D10-K) -> Net-(D25-K)
- D26 pad 2: Net-(D25-A) -> Net-(D10-A)
- D27 pad 1: Net-(D11-K) -> Net-(D25-K)
- D27 pad 2: Net-(D25-A) -> Net-(D11-A)
- D28 pad 1: Net-(D12-K) -> Net-(D25-K)
- D28 pad 2: Net-(D25-A) -> Net-(D12-A)
- D29 pad 1: Net-(D13-K) -> Net-(D25-K)
- D29 pad 2: Net-(D25-A) -> Net-(D13-A)
- D3 pad 1: Net-(D11-K) -> Net-(D1-K)
- D3 pad 2: Net-(D1-A) -> Net-(D11-A)
- D30 pad 1: Net-(D14-K) -> Net-(D25-K)
- D30 pad 2: Net-(D25-A) -> Net-(D14-A)
- D31 pad 1: Net-(D15-K) -> Net-(D25-K)
- D31 pad 2: Net-(D25-A) -> Net-(D15-A)
- D32 pad 1: Net-(D16-K) -> Net-(D25-K)
- D32 pad 2: Net-(D25-A) -> Net-(D16-A)
- D33 pad 1: Net-(D1-K) -> Net-(D33-K)
- D33 pad 2: Net-(D33-A) -> Net-(D1-A)
- D34 pad 1: Net-(D1-K) -> Net-(D33-K)
- D34 pad 2: Net-(D34-A) -> Net-(D10-A)
- D35 pad 1: Net-(D1-K) -> Net-(D33-K)
- D35 pad 2: Net-(D35-A) -> Net-(D11-A)
- D36 pad 1: Net-(D1-K) -> Net-(D33-K)
- D36 pad 2: Net-(D36-A) -> Net-(D12-A)
- D37 pad 1: Net-(D10-K) -> Net-(D33-K)
- D37 pad 2: Net-(D33-A) -> Net-(D13-A)
- D38 pad 1: Net-(D10-K) -> Net-(D33-K)
- D38 pad 2: Net-(D34-A) -> Net-(D14-A)
- D39 pad 1: Net-(D10-K) -> Net-(D33-K)
- D39 pad 2: Net-(D35-A) -> Net-(D15-A)
- D4 pad 1: Net-(D12-K) -> Net-(D1-K)
- D4 pad 2: Net-(D1-A) -> Net-(D12-A)
- D40 pad 1: Net-(D10-K) -> Net-(D33-K)
- D40 pad 2: Net-(D36-A) -> Net-(D16-A)
- D41 pad 1: Net-(D11-K) -> Net-(D41-K)
- D41 pad 2: Net-(D33-A) -> Net-(D1-A)
- D42 pad 1: Net-(D11-K) -> Net-(D41-K)
- D42 pad 2: Net-(D34-A) -> Net-(D10-A)
- D43 pad 1: Net-(D11-K) -> Net-(D41-K)
- D43 pad 2: Net-(D35-A) -> Net-(D11-A)
- D44 pad 1: Net-(D11-K) -> Net-(D41-K)
- D44 pad 2: Net-(D36-A) -> Net-(D12-A)
- D45 pad 1: Net-(D12-K) -> Net-(D41-K)
- D45 pad 2: Net-(D33-A) -> Net-(D13-A)
- D46 pad 1: Net-(D12-K) -> Net-(D41-K)
- D46 pad 2: Net-(D34-A) -> Net-(D14-A)
- D47 pad 1: Net-(D12-K) -> Net-(D41-K)
- D47 pad 2: Net-(D35-A) -> Net-(D15-A)
- D48 pad 1: Net-(D12-K) -> Net-(D41-K)
- D48 pad 2: Net-(D36-A) -> Net-(D16-A)
- D49 pad 1: Net-(D13-K) -> Net-(D49-K)
- D49 pad 2: Net-(D33-A) -> Net-(D1-A)
- D5 pad 1: Net-(D13-K) -> Net-(D1-K)
- D5 pad 2: Net-(D1-A) -> Net-(D13-A)
- D50 pad 1: Net-(D13-K) -> Net-(D49-K)
- D50 pad 2: Net-(D34-A) -> Net-(D10-A)
- D51 pad 1: Net-(D13-K) -> Net-(D49-K)
- D51 pad 2: Net-(D35-A) -> Net-(D11-A)
- D52 pad 1: Net-(D13-K) -> Net-(D49-K)
- D52 pad 2: Net-(D36-A) -> Net-(D12-A)
- D53 pad 1: Net-(D14-K) -> Net-(D49-K)
- D53 pad 2: Net-(D33-A) -> Net-(D13-A)
- D54 pad 1: Net-(D14-K) -> Net-(D49-K)
- D54 pad 2: Net-(D34-A) -> Net-(D14-A)
- D55 pad 1: Net-(D14-K) -> Net-(D49-K)
- D55 pad 2: Net-(D35-A) -> Net-(D15-A)
- D56 pad 1: Net-(D14-K) -> Net-(D49-K)
- D56 pad 2: Net-(D36-A) -> Net-(D16-A)
- D57 pad 1: Net-(D15-K) -> Net-(D57-K)
- D57 pad 2: Net-(D33-A) -> Net-(D1-A)
- D58 pad 1: Net-(D15-K) -> Net-(D57-K)
- D58 pad 2: Net-(D34-A) -> Net-(D10-A)
- D59 pad 1: Net-(D15-K) -> Net-(D57-K)
- D59 pad 2: Net-(D35-A) -> Net-(D11-A)
- D6 pad 1: Net-(D14-K) -> Net-(D1-K)
- D6 pad 2: Net-(D1-A) -> Net-(D14-A)
- D60 pad 1: Net-(D15-K) -> Net-(D57-K)
- D60 pad 2: Net-(D36-A) -> Net-(D12-A)
- D61 pad 1: Net-(D16-K) -> Net-(D57-K)
- D61 pad 2: Net-(D33-A) -> Net-(D13-A)
- D62 pad 1: Net-(D16-K) -> Net-(D57-K)
- D62 pad 2: Net-(D34-A) -> Net-(D14-A)
- D63 pad 1: Net-(D16-K) -> Net-(D57-K)
- D63 pad 2: Net-(D35-A) -> Net-(D15-A)
- D64 pad 1: Net-(D16-K) -> Net-(D57-K)
- D64 pad 2: Net-(D36-A) -> Net-(D16-A)
- D7 pad 1: Net-(D15-K) -> Net-(D1-K)
- D7 pad 2: Net-(D1-A) -> Net-(D15-A)
- D8 pad 1: Net-(D16-K) -> Net-(D1-K)
- D8 pad 2: Net-(D1-A) -> Net-(D16-A)
- D9 pad 1: Net-(D1-K) -> Net-(D10-K)
- D9 pad 2: Net-(D10-A) -> Net-(D1-A)
- RN1 pad 3: Net-(D17-A) -> Net-(D11-A)
- RN1 pad 4: Net-(D25-A) -> Net-(D12-A)
- RN2 pad 1: Net-(D33-A) -> Net-(D13-A)
- RN2 pad 2: Net-(D34-A) -> Net-(D14-A)
- RN2 pad 3: Net-(D35-A) -> Net-(D15-A)
- RN2 pad 4: Net-(D36-A) -> Net-(D16-A)
- RN3 pad 3: Net-(D11-K) -> Net-(D17-K)
- RN3 pad 4: Net-(D12-K) -> Net-(D25-K)
- RN4 pad 1: Net-(D13-K) -> Net-(D33-K)
- RN4 pad 2: Net-(D14-K) -> Net-(D41-K)
- RN4 pad 3: Net-(D15-K) -> Net-(D49-K)
- RN4 pad 4: Net-(D16-K) -> Net-(D57-K)
Routing:
- net Net-(D25-K): track 0.00 -> 26.7 mm
- net Net-(D17-K): track 0.00 -> 26.7 mm
- net Net-(D10-K): track 0.00 -> 26.7 mm
- net Net-(D1-K): track 0.00 -> 26.7 mm
- net Net-(D57-K): track 0.00 -> 26.7 mm
- net Net-(D49-K): track 0.00 -> 26.7 mm
- net Net-(D41-K): track 0.00 -> 26.7 mm
- net Net-(D33-K): track 0.00 -> 26.7 mm
- net LZ7: track 0.00 -> 2.50 mm
- net LZ6: track 0.00 -> 2.50 mm
- net LZ5: track 0.00 -> 2.50 mm
- net LZ4: track 0.00 -> 2.50 mm
- net LZ3: track 0.00 -> 2.50 mm
- net LZ2: track 0.00 -> 2.50 mm
- net LZ1: track 0.00 -> 2.50 mm
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Other:
- board text added: "Z0"
- board text added: "Z1"
- board text added: "Z2"
- board text added: "Z3"
- board text added: "Z4"
- board text added: "Z5"
- board text added: "Z6"
- board text added: "Z7"

Commit message: halb
Parts:
- moved D1 16.5 mm to (223.1, 52.1)
- moved D2 16.5 mm to (223.1, 55.9)
- moved D3 16.5 mm to (223.1, 59.7)
- moved D33 16.5 mm to (223.1, 97.8)
- moved D34 16.5 mm to (223.1, 101.6)
- moved D35 16.5 mm to (223.1, 105.4)
- moved D36 16.5 mm to (223.1, 109.2)
- moved D37 16.5 mm to (223.1, 113.0)
- moved D38 16.5 mm to (223.1, 116.8)
- moved D39 16.5 mm to (223.1, 120.7)
- moved D4 16.5 mm to (223.1, 63.5)
- moved D40 16.5 mm to (223.1, 124.5)
- moved D5 16.5 mm to (223.1, 67.3)
- moved D6 16.5 mm to (223.1, 71.1)
- moved D7 16.5 mm to (223.1, 74.9)
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Routing:
- net Net-(D13-A): track 0.00 -> 54.4 mm, vias 0 -> 8
- net Net-(D14-A): track 0.00 -> 51.8 mm, vias 0 -> 8
- net Net-(D15-A): track 0.00 -> 48.6 mm, vias 0 -> 8
- net Net-(D16-A): track 0.00 -> 45.7 mm, vias 0 -> 8
- net Net-(D10-A): track 0.00 -> 45.4 mm, vias 0 -> 8
- net Net-(D11-A): track 0.00 -> 42.5 mm, vias 0 -> 8
- net Net-(D1-A): track 0.00 -> 41.8 mm, vias 0 -> 2
- net Net-(D12-A): track 0.00 -> 41.4 mm, vias 0 -> 8
- net Net-(D25-K): track 26.7 -> 49.3 mm
- net Net-(D17-K): track 26.7 -> 46.5 mm
- net LS4: track 0.00 -> 19.7 mm
- net Net-(D57-K): track 26.7 -> 45.4 mm
- net LS0: track 0.00 -> 18.1 mm
- net Net-(D10-K): track 26.7 -> 44.1 mm
- net LZ3: track 2.50 -> 18.8 mm
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Other:
- board size 36.8 x 92.7 mm -> 31.1 x 92.7 mm

Commit message: routed
Parts:
- moved RN1 173.4 mm to (57.6, 29.3)
- moved LAMPENSPALTEN1 171.7 mm to (64.2, 67.3)
- moved LAMPENZEILEN1 171.7 mm to (64.2, 112.9)
- moved RN4 170.9 mm to (57.6, 112.5)
- moved RN3 170.8 mm to (57.6, 75.6)
- moved RN2 170.7 mm to (57.6, 69.3)
- moved D33 168.9 mm to (55.0, 81.3)
- moved D34 168.9 mm to (55.0, 85.1)
- moved D35 168.9 mm to (55.0, 88.9)
- moved D36 168.9 mm to (55.0, 92.7)
- moved D37 168.9 mm to (55.0, 96.5)
- moved D38 168.9 mm to (55.0, 100.3)
- moved D39 168.9 mm to (55.0, 104.1)
- moved D40 168.9 mm to (55.0, 108.0)
- moved D41 168.9 mm to (51.2, 81.3)
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Routing:
- net Net-(D12-A): track 41.4 -> 119.0 mm
- net Net-(D11-A): track 42.5 -> 116.5 mm
- net Net-(D1-A): track 41.8 -> 112.6 mm
- net Net-(D10-A): track 45.4 -> 113.7 mm
- net Net-(D13-A): track 54.4 -> 115.2 mm
- net Net-(D14-A): track 51.8 -> 112.1 mm
- net Net-(D15-A): track 48.6 -> 108.7 mm
- net Net-(D16-A): track 45.7 -> 105.4 mm
- net LS3: track 9.27 -> 19.2 mm
- net LS0: track 18.1 -> 8.99 mm
- net LS2: track 11.0 -> 15.4 mm
- net Net-(D10-K): track 44.1 -> 40.7 mm
- net Net-(D1-K): track 41.3 -> 38.0 mm
- net Net-(D17-K): track 46.5 -> 43.4 mm
- net LS1: track 14.2 -> 11.2 mm
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Other:
- board size 31.1 x 92.7 mm -> 29.8 x 91.4 mm
- board text added: "Lampen Tester"
- board text added: "S0"
- board text added: "S1"
- board text added: "S2"
- board text added: "S3"
- board text added: "S4"
- board text added: "S5"
- board text added: "S6"
- board text added: "S7"
