File: Maschinenplatine/Maschinenplatine.kicad_sch (KiCad schematic)
At the start: 14 parts, among them IC1 4069, J1 Hauptmaschine, U1 4070, U2 4098

Commit message: motor1
Parts:
- added C14: 1uF, symbol Device:C_Polarized_Small
- added C19: 10uF, symbol Device:C_Polarized_Small
- added D10, D11, D8: ZPD 9,1, symbol Device:D_Zener
- added D12, D9: 1N4148, Diode_THT:D_DO-35_SOD27_P7.62mm_Horizontal, symbol Diode:1N4148
- added IC5: HEF4093B, symbol 4xxx:HEF4093B
- added LA1: Scheibe 1, symbol Device:Lamp
- added LA2, LA4: 6V/2W, symbol Device:Lamp
- added LA3: Scheibe 2, symbol Device:Lamp
- added LA5: Scheibe 3, symbol Device:Lamp
- added Lichtschr.1, Lichtschr.2, Lichtschr.3: ITR9608-F, OptoDevice:Everlight_ITR9608-F, symbol Sensor_Proximity:ITR9608-F
- added M1: Conn_01x04, symbol Connector_Generic:Conn_01x04
- added R11, R27, R4: 100K, symbol Device:R
- added R12: 10R, symbol Device:R
- added R14: 1K-1/2W, symbol Device:R
- added R15: 47R, symbol Device:R
- added R16: 470R, symbol Device:R
- added R2: 10R/7W, symbol Device:R
- added R3, R49, R51: 330R, symbol Device:R
- added T10: BC546, Package_TO_SOT_THT:TO-92_Inline, symbol Transistor_BJT:BC546
- added T11, T12: BSS97, symbol Transistor_FET:Q_NMOS_GDS
- added T6: BC327, Package_TO_SOT_THT:TO-92_Inline, symbol Transistor_BJT:BC327
- added T7: BC337, Package_TO_SOT_THT:TO-92_Inline, symbol Transistor_BJT:BC337
- added T9: BS170, Package_TO_SOT_THT:TO-92_Inline, symbol Transistor_FET:BS170
- renumbered U1 to IC2, U2 to IC3
Connections:
- net +12V: now also Lichtschr.1.1, Lichtschr.1.3, Lichtschr.2.1, Lichtschr.2.3, Lichtschr.3.1, Lichtschr.3.3
- net +20V: now also M1.2 (Pin_2), M1.4 (Pin_4)
- net GND: now also IC1.7 (VSS), IC2.7 (VSS), IC3.8 (VSS), D8.2 (A), IC5.7 (GND), R11.2, R3.2, R4.2, R49.2, R51.2, T11.3 (S), T6.1 (C), T9.3 (S)
- net M1A: no longer C4.1, J1.19 (Pin_19), RM11.6 (R6.1)
- net VDD: now also R27.1, T7.1 (C)
- net at IC2.10: now also R11.1, T6.2 (B), T7.2 (B)
- net at IC2.6, IC2.8: now also IC5.10
- net at IC3.14 (Rx2_Cx2): now also C19.1, R27.2
- net at IC3.15 (Cx2): now also C19.2
- net at IC3.9 (~{Q2}): now also IC5.8
- net M2A: now reaches C3.1, J1.18 (Pin_18), RM11.5 (R5.1)
- net M2B: now reaches C2.1, J1.17 (Pin_17), RM11.4 (R4.1)
- net LiS3: now reaches J1.2 (Pin_2)
- net LiS3: now also Lichtschr.3.4
- net LiS2: now reaches J1.3 (Pin_3)
- net LiS2: now also Lichtschr.2.4
- net LiS1: now reaches J1.4 (Pin_4)
- net LiS1: now also Lichtschr.1.4
- net LZ6: now reaches J1.7 (Pin_7)
- net LZ6: now also LA1.2 (+), LA2.2 (+), LA3.2 (+), LA4.2 (+), LA5.2 (+)
- net at IC2.4: now also R4.1
- net at D2.1 (K): now also LA3.1 (-), LA4.1 (-)
- net at D3.1 (K): now also LA5.1 (-)
- net at D1.1 (K): now also LA1.1 (-), LA2.1 (-)
- new net: D9.1 (K), R12.1, R14.1, T10.2 (B)
- new net: D11.1 (K), D9.2 (A), T10.3 (E), T12.1 (G)
- new net: R12.2, T9.1 (D)
- new net: R15.2, T6.3 (E), T7.3 (E), T9.2 (G)
- new net: D12.1 (K), R16.1
- new net: D12.2 (A), T12.2 (D)
- new net: C14.1, R14.2, R16.2, T10.1 (C)
- new net: C14.2, D10.1 (K), R2.2, T11.2 (D), T12.3 (S)
- new net: D10.2 (A), D11.2 (A)
- new net: Lichtschr.3.2, R51.1
- new net: M1.3 (Pin_3), R2.1
- new net: D8.1 (K), R15.1, T11.1 (G)
- new net: Lichtschr.1.2, R3.1
- new net: Lichtschr.2.2, R49.1
- new net M1B: C4.1, J1.19 (Pin_19), RM11.6 (R6.1)
Other:
- moved on the sheet: C1, C2, C3, C4, C5, C6, D1, D2, D3, IC1A, IC1B, IC1C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
